Commit message: Meshes added

File: src/mobile_manipulator/model/test.urdf (robot description, URDF)
Before this commit: robot mobile_manipulator, 11 links, 10 joints
Links:
- link WristPitch: geometry collision box size=0.032 0.04 0.05; visual mesh filename=package://mobile_manipulator/meshes/AX-12_18A - dynamixel_A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 scale=0.001 0.001 0.001
- link WristRoll: geometry collision box size=0.032 0.04 0.05; visual mesh filename=package://mobile_manipulator/meshes/AX-12_18A - dynamixel_A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 scale=0.001 0.001 0.001
- link base_link: geometry collision box size=0.041 0.0402 0.0611; visual mesh filename=package://mobile_manipulator/meshes/dynamixel_x64series.stl scale=0.001 0.001 0.001
- link elbow: geometry collision box size=0.041 0.0402 0.0611; visual mesh filename=package://mobile_manipulator/meshes/dynamixel_x64series.stl scale=0.001 0.001 0.001
- link end_effector: geometry collision mesh filename=package://mobile_manipulator/meshes/FR05-H101K.stl scale=0.001 0.001 0.001; visual mesh filename=package://mobile_manipulator/meshes/FR05-H101K.stl scale=0.001 0.001 0.001
- link link1Bracket: geometry collision mesh filename=package://mobile_manipulator/meshes/FR05-H101K.stl scale=0.001 0.001 0.001; visual mesh filename=package://mobile_manipulator/meshes/FR05-H101K.stl scale=0.001 0.001 0.001
- link link2Bracket: geometry collision mesh filename=package://mobile_manipulator/meshes/FR05-H101K.stl scale=0.001 0.001 0.001; visual mesh filename=package://mobile_manipulator/meshes/FR05-H101K.stl scale=0.001 0.001 0.001
- link link3Bracket: geometry collision mesh filename=package://mobile_manipulator/meshes/FR05-H101K.stl scale=0.001 0.001 0.001; visual mesh filename=package://mobile_manipulator/meshes/FR05-H101K.stl scale=0.001 0.001 0.001
- link shoulder1: geometry collision box size=0.041 0.0402 0.0611; visual mesh filename=package://mobile_manipulator/meshes/dynamixel_x64series.stl scale=0.001 0.001 0.001
