Commit message: Mesh files Added

File: src/mobile_manipulator/model/mobile_manipulator.xacro (robot description, xacro)
@@ -22,5 +22,5 @@
     <origin xyz="${trans}" rpy="${rpy}"/>
     <geometry>
-      <mesh filename="package://avitra_description/meshes/dynamixel_x64series.stl" scale="0.001 0.001 0.001"/>
+      <mesh filename="package://mobile_manipulator/meshes/dynamixel_x64series.stl" scale="0.001 0.001 0.001"/>
     </geometry>
     <material name="white"/>
@@ -46,5 +46,5 @@
     <origin xyz="${trans}" rpy="${rpy}"/>
     <geometry>
-      <mesh filename="package://avitra_description/meshes/AX-12_18A - dynamixel_AXseries-1.stl" scale="0.001 0.001 0.001"/>
+      <mesh filename="package://mobile_manipulator/meshes/AX-12_18A - dynamixel_AXseries-1.stl" scale="0.001 0.001 0.001"/>
     </geometry>
     <material name="white"/>
@@ -70,5 +70,5 @@
     <origin xyz="${trans}" rpy="${rpy}"/>
     <geometry>
-      <mesh filename="package://avitra_description/meshes/FR05-H101K.stl" scale="0.001 0.001 0.001" />
+      <mesh filename="package://mobile_manipulator/meshes/FR05-H101K.stl" scale="0.001 0.001 0.001" />
     </geometry>
     <material name="white"/>
@@ -79,5 +79,5 @@
       <origin xyz="${trans}" rpy="${rpy}"/>
       <geometry>
-        <mesh filename="package://avitra_description/meshes/FR05-H101K.stl" scale="0.001 0.001 0.001"/>
+        <mesh filename="package://mobile_manipulator/meshes/FR05-H101K.stl" scale="0.001 0.001 0.001"/>
       </geometry>
     </collision>
@@ -94,5 +94,5 @@
     <origin xyz="${trans}" rpy="${rpy}"/>
     <geometry>
-      <mesh filename="package://avitra_description/meshes/FR05-H101K.stl" scale="0.001 0.001 0.001" />
+      <mesh filename="package://mobile_manipulator/meshes/FR05-H101K.stl" scale="0.001 0.001 0.001" />
     </geometry>
     <material name="white"/>
@@ -103,5 +103,5 @@
       <origin xyz="${trans}" rpy="${rpy}"/>
       <geometry>
-        <mesh filename="package://avitra_description/meshes/FR05-H101K.stl" scale="0.001 0.001 0.001"/>
+        <mesh filename="package://mobile_manipulator/meshes/FR05-H101K.stl" scale="0.001 0.001 0.001"/>
       </geometry>
     </collision>

Commit message: Removed Numerical Link names

File: src/mobile_manipulator/model/mobile_manipulator.xacro (robot description, xacro)
@@ -201,13 +201,13 @@
     <xacro:BracketCollision trans="0 0 0" rpy="3.14 0 1.57"/>
   </link>
-  <xacro:Revjoint id="1" trans="0 0 0" rpy="0 0 0" parent="base_link" child="link1Bracket" axis="0 0 1" l="-1.57" u="1.57" v="1.0"/>
-  <xacro:Revjoint id="2" trans="0 0 0.0636" rpy="0 0 0" parent="link1Bracket" child="shoulder1" axis="1 0 0" l="-1.57" u="1.57" v="1.0"/>
+  <xacro:Revjoint id="one" trans="0 0 0" rpy="0 0 0" parent="base_link" child="link1Bracket" axis="0 0 1" l="-1.57" u="1.57" v="1.0"/>
+  <xacro:Revjoint id="two" trans="0 0 0.0636" rpy="0 0 0" parent="link1Bracket" child="shoulder1" axis="1 0 0" l="-1.57" u="1.57" v="1.0"/>
   <xacro:FxdJoint id="s1_l2" parent="shoulder1" child="link2"/>
   <xacro:FxdJoint id="l2_l2B" parent="link2" child="link2Bracket"/>
-  <xacro:Revjoint id="3" trans="0 0 ${0.0867+(length)}" rpy="0 0 0" parent="link2Bracket" child="elbow" axis="1 0 0" l="-1.57" u="3.14" v="1.0"/>
+  <xacro:Revjoint id="three" trans="0 0 ${0.0867+(length)}" rpy="0 0 0" parent="link2Bracket" child="elbow" axis="1 0 0" l="-1.57" u="3.14" v="1.0"/>
   <xacro:FxdJoint id="e_l3" parent="elbow" child="link3"/>
   <xacro:FxdJoint id="l3_l3B" parent="link3" child="link3Bracket"/>
-  <xacro:Revjoint id="4" trans="0 0 ${0.0867+length}" rpy="0 0 0" parent="link3Bracket" child="WristPitch" axis="1 0 0" l="-1.57" u="1.57" v="1.0"/>
+  <xacro:Revjoint id="four" trans="0 0 ${0.0867+length}" rpy="0 0 0" parent="link3Bracket" child="WristPitch" axis="1 0 0" l="-1.57" u="1.57" v="1.0"/>
   <xacro:FxdJoint id="WP_WR" parent="WristPitch" child="WristRoll"/>
-  <xacro:Revjoint id="5" trans="0 0.015 0.0785" rpy="0 0 0" parent="WristRoll" child="end_effector" axis="0 0 1" l="-3.14" u="3.14" v="1.0"/>
+  <xacro:Revjoint id="five" trans="0 0.015 0.0785" rpy="0 0 0" parent="WristRoll" child="end_effector" axis="0 0 1" l="-3.14" u="3.14" v="1.0"/>
 </robot>

File: src/mobile_manipulator/model/test.urdf (robot description, URDF)
Before this commit: robot mobile_manipulator, 11 links, 10 joints
Joints:
- removed joint 1
- removed joint 2
- removed joint 3
- removed joint 4
- removed joint 5
- added joint five: type revolute, parent WristRoll, child end_effector, origin xyz=0 0.015 0.0785 rpy=0 0 0, axis 0 0 1, limit lower=-3.14 upper=3.14 effort=30 velocity=1.0
- added joint four: type revolute, parent link3Bracket, child WristPitch, origin xyz=0 0 0.2567 rpy=0 0 0, axis 1 0 0, limit lower=-1.57 upper=1.57 effort=30 velocity=1.0
- added joint one: type revolute, parent base_link, child link1Bracket, origin xyz=0 0 0 rpy=0 0 0, axis 0 0 1, limit lower=-1.57 upper=1.57 effort=30 velocity=1.0
- added joint three: type revolute, parent link2Bracket, child elbow, origin xyz=0 0 0.2567 rpy=0 0 0, axis 1 0 0, limit lower=-1.57 upper=3.14 effort=30 velocity=1.0
- added joint two: type revolute, parent link1Bracket, child shoulder1, origin xyz=0 0 0.0636 rpy=0 0 0, axis 1 0 0, limit lower=-1.57 upper=1.57 effort=30 velocity=1.0

Commit message: Bracket dimesions changed

File: src/mobile_manipulator/model/mobile_manipulator.xacro (robot description, xacro)
@@ -10,5 +10,5 @@
 <xacro:property name="AXWidth" value="0.032"/>
 <xacro:property name="AXDepth" value="0.04"/>
-<xacro:property name="length" value="0.17"/>
+<xacro:property name="length" value="0.096"/>
 <xacro:macro name="MXInertial" params="trans rpy">
   <inertial>
@@ -94,5 +94,5 @@
     <origin xyz="${trans}" rpy="${rpy}"/>
     <geometry>
-      <mesh filename="package://mobile_manipulator/meshes/FR05-H101K.stl" scale="0.001 0.001 0.001" />
+      <mesh filename="package://mobile_manipulator/meshes/F4.stl" scale="0.001 0.001 0.001" />
     </geometry>
     <material name="white"/>
@@ -103,5 +103,5 @@
       <origin xyz="${trans}" rpy="${rpy}"/>
       <geometry>
-        <mesh filename="package://mobile_manipulator/meshes/FR05-H101K.stl" scale="0.001 0.001 0.001"/>
+        <mesh filename="package://mobile_manipulator/meshes/F4.stl" scale="0.001 0.001 0.001"/>
       </geometry>
     </collision>
@@ -182,7 +182,7 @@
   </link>
   <link name="link3Bracket">
-    <xacro:BracketInertial trans="0 0 ${0.0481+length}" rpy="0 3.14 0"/>
-    <xacro:BracketVisual trans="0 0 ${0.0481+length}" rpy="0 3.14 0"/>
-    <xacro:BracketCollision trans="0 0 ${0.0481+length}" rpy="0 3.14 0"/>
+    <xacro:AxBracketInertial trans="0 0 ${0.0988+length}" rpy="1.57 0 1.57"/>
+    <xacro:AxBracketVisual trans="0 0 ${0.0988+length}" rpy="1.57 0 1.57"/>
+    <xacro:AxBracketCollision trans="0 0 ${0.0988+length}" rpy="1.57 0 1.57"/>
   </link>
   <link name="WristPitch">
@@ -205,8 +205,8 @@
   <xacro:FxdJoint id="s1_l2" parent="shoulder1" child="link2"/>
   <xacro:FxdJoint id="l2_l2B" parent="link2" child="link2Bracket"/>
-  <xacro:Revjoint id="three" trans="0 0 ${0.0867+(length)}" rpy="0 0 0" parent="link2Bracket" child="elbow" axis="1 0 0" l="-1.57" u="3.14" v="1.0"/>
+  <xacro:Revjoint id="three" trans="0 0 ${0.0867+(length)}" rpy="0 0 0" parent="link2Bracket" child="elbow" axis="1 0 0" l="-1.57" u="1.57" v="1.0"/>
   <xacro:FxdJoint id="e_l3" parent="elbow" child="link3"/>
   <xacro:FxdJoint id="l3_l3B" parent="link3" child="link3Bracket"/>
-  <xacro:Revjoint id="four" trans="0 0 ${0.0867+length}" rpy="0 0 0" parent="link3Bracket" child="WristPitch" axis="1 0 0" l="-1.57" u="1.57" v="1.0"/>
+  <xacro:Revjoint id="four" trans="0 0 ${0.0988+length}" rpy="0 0 0" parent="link3Bracket" child="WristPitch" axis="1 0 0" l="-1.57" u="1.57" v="1.0"/>
   <xacro:FxdJoint id="WP_WR" parent="WristPitch" child="WristRoll"/>
   <xacro:Revjoint id="five" trans="0 0.015 0.0785" rpy="0 0 0" parent="WristRoll" child="end_effector" axis="0 0 1" l="-3.14" u="3.14" v="1.0"/>

File: src/mobile_manipulator/model/test.urdf (robot description, URDF)
Before this commit: robot mobile_manipulator, 11 links, 10 joints
Links:
- link link2: mass 0.00085 -> 0.00048; geometry collision box size=0.04 0.04 0.096; visual box size=0.04 0.04 0.096
- link link3: mass 0.00085 -> 0.00048; geometry collision box size=0.04 0.04 0.096; visual box size=0.04 0.04 0.096
- link link3Bracket: geometry collision mesh filename=package://mobile_manipulator/meshes/F4.stl scale=0.001 0.001 0.001; visual mesh filename=package://mobile_manipulator/meshes/F4.stl scale=0.001 0.001 0.001
Joints:
- joint four: origin xyz=0 0 0.2567 rpy=0 0 0 -> xyz=0 0 0.1948 rpy=0 0 0
- joint three: limit lower=-1.57 upper=3.14 effort=30 velocity=1.0 -> lower=-1.57 upper=1.57 effort=30 velocity=1.0; origin xyz=0 0 0.2567 rpy=0 0 0 -> xyz=0 0 0.1827 rpy=0 0 0

Commit message: Kinematic Solver changed in config file

File: src/mobile_manipulator/model/mobile_manipulator.xacro (robot description, xacro)
@@ -201,5 +201,5 @@
     <xacro:BracketCollision trans="0 0 0" rpy="3.14 0 1.57"/>
   </link>
-  <xacro:Revjoint id="one" trans="0 0 0" rpy="0 0 0" parent="base_link" child="link1Bracket" axis="0 0 1" l="-1.57" u="1.57" v="1.0"/>
+  <xacro:Revjoint id="one" trans="0 0 0" rpy="0 0 0" parent="base_link" child="link1Bracket" axis="0 0 1" l="-3.14" u="3.14" v="1.0"/>
   <xacro:Revjoint id="two" trans="0 0 0.0636" rpy="0 0 0" parent="link1Bracket" child="shoulder1" axis="1 0 0" l="-1.57" u="1.57" v="1.0"/>
   <xacro:FxdJoint id="s1_l2" parent="shoulder1" child="link2"/>

File: src/mobile_manipulator/model/test.urdf (robot description, URDF)
Before this commit: robot mobile_manipulator, 11 links, 10 joints
Joints:
- joint one: limit lower=-1.57 upper=1.57 effort=30 velocity=1.0 -> lower=-3.14 upper=3.14 effort=30 velocity=1.0

Commit message: trash commit for atharv

File: src/mobile_manipulator/model/mobile_manipulator.xacro (robot description, xacro)
@@ -146,50 +146,50 @@
     </joint>
 </xacro:macro>
-  <link name="base_link">
+  <link name="shoulder_yaw_motor">
     <xacro:MXInertial trans="0 0 0" rpy="0 0 0 "/>
     <xacro:MXVisual trans="0 0 0" rpy="0 0 0 "/>
     <xacro:MXCollision trans="0 0 0" rpy="0 0 0"/>
   </link>
-  <link name="link1Bracket">
+  <link name="shoulder_bracket">
     <xacro:BracketInertial trans="0 0 0.025" rpy="0 3.14 0 "/>
     <xacro:BracketVisual trans="0 0 0.025" rpy="0 3.14 0 "/>
     <xacro:BracketCollision trans="0 0 0.025" rpy="0 3.14 0 "/>
   </link>
-  <link name="shoulder1">
+  <link name="shoulder_pitch_motor">
     <xacro:MXInertial trans="0 0 0" rpy="1.57 -3.14 1.57"/>
     <xacro:MXVisual trans="0 0 0" rpy="1.57 -3.14 1.57"/>
     <xacro:MXCollision trans="0 0 0" rpy="1.57 -3.14 1.57"/>
   </link>
-  <link name="link2">
+  <link name="biscep">
     <xacro:LinkInertial trans="0 0 ${0.0481+(length/2)}" rpy="0 0 0" />
     <xacro:LinkVisual trans="0 0 ${0.0481+(length/2)}" rpy="0 0 0" />
     <xacro:LinkCollision trans="0 0 ${0.0481+(length/2)}" rpy="0 0 0" />
   </link>
-  <link name="link2Bracket">
+  <link name="elbow_bracket">
     <xacro:BracketInertial trans="0 0 ${0.0481+length}" rpy="0 3.14 0"/>
     <xacro:BracketVisual trans="0 0 ${0.0481+length}" rpy="0 3.14 0"/>
     <xacro:BracketCollision trans="0 0 ${0.0481+length}" rpy="0 3.14 0"/>
   </link>
-  <link name="elbow">
+  <link name="elbow_motor">
     <xacro:MXInertial trans="0 0 0" rpy="1.57 0 0"/>
     <xacro:MXVisual trans="0 0 0" rpy="1.57 3.14 -1.57"/>
     <xacro:MXCollision trans="0 0 0" rpy="1.57 0 0"/>
   </link>
-  <link name="link3">
+  <link name="forearm">
     <xacro:LinkInertial trans="0 0 ${0.0481+(length/2)}" rpy="0 0 0" />
     <xacro:LinkVisual trans="0 0 ${0.0481+(length/2)}" rpy="0 0 0" />
     <xacro:LinkCollision trans="0 0 ${0.0481+(length/2)}" rpy="0 0 0" />
   </link>
-  <link name="link3Bracket">
+  <link name="wrist_bracket">
     <xacro:AxBracketInertial trans="0 0 ${0.0988+length}" rpy="1.57 0 1.57"/>
     <xacro:AxBracketVisual trans="0 0 ${0.0988+length}" rpy="1.57 0 1.57"/>
     <xacro:AxBracketCollision trans="0 0 ${0.0988+length}" rpy="1.57 0 1.57"/>
   </link>
-  <link name="WristPitch">
+  <link name="wrist_pitch_motor">
     <xacro:AXInertial trans="0 0 0" rpy="-1.57 0 -1.57"/>
     <xacro:AXVisual trans="0. 0 0" rpy="-1.57 0 -1.57"/>
     <xacro:AXCollision trans="0 0 0" rpy="-1.57 0 -1.57"/>
   </link>
-  <link name="WristRoll">
+  <link name="wrist_roll_motor">
     <xacro:AXInertial trans="0 0.015 0.0585" rpy="0 0 0"/>
     <xacro:AXVisual trans="0 0.015 0.0585" rpy="0 0 0"/>
@@ -201,13 +201,13 @@
     <xacro:BracketCollision trans="0 0 0" rpy="3.14 0 1.57"/>
   </link>
-  <xacro:Revjoint id="one" trans="0 0 0" rpy="0 0 0" parent="base_link" child="link1Bracket" axis="0 0 1" l="-3.14" u="3.14" v="1.0"/>
-  <xacro:Revjoint id="two" trans="0 0 0.0636" rpy="0 0 0" parent="link1Bracket" child="shoulder1" axis="1 0 0" l="-1.57" u="1.57" v="1.0"/>
-  <xacro:FxdJoint id="s1_l2" parent="shoulder1" child="link2"/>
-  <xacro:FxdJoint id="l2_l2B" parent="link2" child="link2Bracket"/>
-  <xacro:Revjoint id="three" trans="0 0 ${0.0867+(length)}" rpy="0 0 0" parent="link2Bracket" child="elbow" axis="1 0 0" l="-1.57" u="1.57" v="1.0"/>
-  <xacro:FxdJoint id="e_l3" parent="elbow" child="link3"/>
-  <xacro:FxdJoint id="l3_l3B" parent="link3" child="link3Bracket"/>
-  <xacro:Revjoint id="four" trans="0 0 ${0.0988+length}" rpy="0 0 0" parent="link3Bracket" child="WristPitch" axis="1 0 0" l="-1.57" u="1.57" v="1.0"/>
-  <xacro:FxdJoint id="WP_WR" parent="WristPitch" child="WristRoll"/>
-  <xacro:Revjoint id="five" trans="0 0.015 0.0785" rpy="0 0 0" parent="WristRoll" child="end_effector" axis="0 0 1" l="-3.14" u="3.14" v="1.0"/>
+  <xacro:Revjoint id="shoulder_yaw" trans="0 0 0" rpy="0 0 0" parent="shoulder_yaw_motor" child="shoulder_bracket" axis="0 0 1" l="-3.14" u="3.14" v="1.0"/>
+  <xacro:Revjoint id="shoulder_pitch" trans="0 0 0.0636" rpy="0 0 0" parent="shoulder_bracket" child="shoulder_pitch_motor" axis="1 0 0" l="-1.57" u="1.57" v="1.0"/>
+  <xacro:FxdJoint id="s1_l2" parent="shoulder_pitch_motor" child="biscep"/>
+  <xacro:FxdJoint id="l2_l2B" parent="biscep" child="elbow_bracket"/>
+  <xacro:Revjoint id="elbow" trans="0 0 ${0.0867+(length)}" rpy="0 0 0" parent="elbow_bracket" child="elbow_motor" axis="1 0 0" l="-1.57" u="1.57" v="1.0"/>
+  <xacro:FxdJoint id="e_l3" parent="elbow_motor" child="forearm"/>
+  <xacro:FxdJoint id="l3_l3B" parent="forearm" child="wrist_bracket"/>
+  <xacro:Revjoint id="wrist_pitch" trans="0 0 ${0.0988+length}" rpy="0 0 0" parent="wrist_bracket" child="wrist_pitch_motor" axis="1 0 0" l="-1.57" u="1.57" v="1.0"/>
+  <xacro:FxdJoint id="WP_WR" parent="wrist_pitch_motor" child="wrist_roll_motor"/>
+  <xacro:Revjoint id="wrist_roll" trans="0 0.015 0.0785" rpy="0 0 0" parent="wrist_roll_motor" child="end_effector" axis="0 0 1" l="-3.14" u="3.14" v="1.0"/>
 </robot>
