Commit message: Adding Gripper in xacro

File: src/mobile_manipulator/model/mobile_manipulator.xacro (robot description, xacro)
@@ -11,4 +11,5 @@
 <xacro:property name="AXDepth" value="0.04"/>
 <xacro:property name="length" value="0.096"/>
+<!--XACROS-->
 <xacro:macro name="MXInertial" params="trans rpy">
   <inertial>
@@ -128,4 +129,124 @@
       <geometry>
         <box size="0.04 0.04 ${length}"/>
+      </geometry>
+    </collision>
+</xacro:macro>
+<xacro:macro name="F10Inertial" params="trans rpy">
+  <inertial>
+    <origin xyz="${trans}" rpy="${rpy}"/>
+    <mass value="0.00712" />
+    <inertia ixx="0.00000174511" iyy="0.00000379922" ixz="0.0" ixy="0.0" iyz="0.0" izz="0.00000357521" />
+  </inertial>
+</xacro:macro>
+<xacro:macro name="F10Visual" params="trans rpy">
+  <visual>
+    <origin xyz="${trans}" rpy="${rpy}"/>
+    <geometry>
+      <mesh filename="package://mobile_manipulator/meshes/F10.stl" scale="0.001 0.001 0.001" />
+    </geometry>
+    <material name="white"/>
+  </visual>
+</xacro:macro>
+<xacro:macro name="F10Collision" params="trans rpy">
+    <collision>
+      <origin xyz="${trans}" rpy="${rpy}"/>
+      <geometry>
+        <mesh filename="package://mobile_manipulator/meshes/F10.stl" scale="0.001 0.001 0.001"/>
+      </geometry>
+    </collision>
+</xacro:macro>
+ <xacro:macro name="F9Inertial" params="trans rpy">
+  <inertial>
+    <origin xyz="${trans}" rpy="${rpy}"/>
+    <mass value="0.00712" />
+    <inertia ixx="0.00000174511" iyy="0.00000379922" ixz="0.0" ixy="0.0" iyz="0.0" izz="0.00000357521" />
+  </inertial>
+</xacro:macro>
+<xacro:macro name="F9Visual" params="trans rpy">
+  <visual>
+    <origin xyz="${trans}" rpy="${rpy}"/>
+    <geometry>
+      <mesh filename="package://mobile_manipulator/meshes/F9.stl" scale="0.001 0.001 0.001" />
+    </geometry>
+    <material name="white"/>
+  </visual>
+</xacro:macro>
+<xacro:macro name="F9Collision" params="trans rpy">
+    <collision>
+      <origin xyz="${trans}" rpy="${rpy}"/>
+      <geometry>
+        <mesh filename="package://mobile_manipulator/meshes/F9.stl" scale="0.001 0.001 0.001"/>
+      </geometry>
+    </collision>
+</xacro:macro>
+<xacro:macro name="F11Inertial" params="trans rpy">
+  <inertial>
+    <origin xyz="${trans}" rpy="${rpy}"/>
+    <mass value="0.00712" />
+    <inertia ixx="0.00000174511" iyy="0.00000379922" ixz="0.0" ixy="0.0" iyz="0.0" izz="0.00000357521" />
+  </inertial>
+</xacro:macro>
+<xacro:macro name="F11Visual" params="trans rpy">
+  <visual>
+    <origin xyz="${trans}" rpy="${rpy}"/>
+    <geometry>
+      <mesh filename="package://mobile_manipulator/meshes/F11.stl" scale="0.001 0.001 0.001" />
+    </geometry>
+    <material name="white"/>
+  </visual>
+</xacro:macro>
+<xacro:macro name="F11Collision" params="trans rpy">
+    <collision>
+      <origin xyz="${trans}" rpy="${rpy}"/>
+      <geometry>
+        <mesh filename="package://mobile_manipulator/meshes/F11.stl" scale="0.001 0.001 0.001"/>
+      </geometry>
+    </collision>
+</xacro:macro>
+<xacro:macro name="F3Inertial" params="trans rpy">
+  <inertial>
+    <origin xyz="${trans}" rpy="${rpy}"/>
+    <mass value="0.00712" />
+    <inertia ixx="0.00000174511" iyy="0.00000379922" ixz="0.0" ixy="0.0" iyz="0.0" izz="0.00000357521" />
+  </inertial>
+</xacro:macro>
+<xacro:macro name="F3Visual" params="trans rpy">
+  <visual>
+    <origin xyz="${trans}" rpy="${rpy}"/>
+    <geometry>
+      <mesh filename="package://mobile_manipulator/meshes/F3.stl" scale="0.001 0.001 0.001" />
+    </geometry>
+    <material name="white"/>
+  </visual>
+</xacro:macro>
+<xacro:macro name="F3Collision" params="trans rpy">
+    <collision>
+      <origin xyz="${trans}" rpy="${rpy}"/>
+      <geometry>
+        <mesh filename="package://mobile_manipulator/meshes/F3.stl" scale="0.001 0.001 0.001"/>
+      </geometry>
+    </collision>
+</xacro:macro>
+<xacro:macro name="F6Inertial" params="trans rpy">
+  <inertial>
+    <origin xyz="${trans}" rpy="${rpy}"/>
+    <mass value="0.00712" />
+    <inertia ixx="0.00000174511" iyy="0.00000379922" ixz="0.0" ixy="0.0" iyz="0.0" izz="0.00000357521" />
+  </inertial>
+</xacro:macro>
+<xacro:macro name="F6Visual" params="trans rpy">
+  <visual>
+    <origin xyz="${trans}" rpy="${rpy}"/>
+    <geometry>
+      <mesh filename="package://mobile_manipulator/meshes/F6.stl" scale="0.001 0.001 0.001" />
+    </geometry>
+    <material name="white"/>
+  </visual>
+</xacro:macro>
+<xacro:macro name="F6Collision" params="trans rpy">
+    <collision>
+      <origin xyz="${trans}" rpy="${rpy}"/>
+      <geometry>
+        <mesh filename="package://mobile_manipulator/meshes/F6.stl" scale="0.001 0.001 0.001"/>
       </geometry>
     </collision>
@@ -146,68 +267,112 @@
     </joint>
 </xacro:macro>
-  <link name="shoulder_yaw_motor">
+<!--LINKS-->
+<link name="shoulder_yaw_motor">
     <xacro:MXInertial trans="0 0 0" rpy="0 0 0 "/>
     <xacro:MXVisual trans="0 0 0" rpy="0 0 0 "/>
     <xacro:MXCollision trans="0 0 0" rpy="0 0 0"/>
-  </link>
-  <link name="shoulder_bracket">
+</link>
+<link name="shoulder_bracket">
     <xacro:BracketInertial trans="0 0 0.025" rpy="0 3.14 0 "/>
     <xacro:BracketVisual trans="0 0 0.025" rpy="0 3.14 0 "/>
     <xacro:BracketCollision trans="0 0 0.025" rpy="0 3.14 0 "/>
-  </link>
-  <link name="shoulder_pitch_motor">
+</link>
+<link name="shoulder_pitch_motor">
     <xacro:MXInertial trans="0 0 0" rpy="1.57 -3.14 1.57"/>
     <xacro:MXVisual trans="0 0 0" rpy="1.57 -3.14 1.57"/>
     <xacro:MXCollision trans="0 0 0" rpy="1.57 -3.14 1.57"/>
-  </link>
-  <link name="biscep">
+</link>
+<link name="biscep">
     <xacro:LinkInertial trans="0 0 ${0.0481+(length/2)}" rpy="0 0 0" />
     <xacro:LinkVisual trans="0 0 ${0.0481+(length/2)}" rpy="0 0 0" />
     <xacro:LinkCollision trans="0 0 ${0.0481+(length/2)}" rpy="0 0 0" />
-  </link>
-  <link name="elbow_bracket">
+</link>
+<link name="elbow_bracket">
     <xacro:BracketInertial trans="0 0 ${0.0481+length}" rpy="0 3.14 0"/>
     <xacro:BracketVisual trans="0 0 ${0.0481+length}" rpy="0 3.14 0"/>
     <xacro:BracketCollision trans="0 0 ${0.0481+length}" rpy="0 3.14 0"/>
-  </link>
-  <link name="elbow_motor">
+</link>
+<link name="elbow_motor">
     <xacro:MXInertial trans="0 0 0" rpy="1.57 0 0"/>
     <xacro:MXVisual trans="0 0 0" rpy="1.57 3.14 -1.57"/>
     <xacro:MXCollision trans="0 0 0" rpy="1.57 0 0"/>
-  </link>
-  <link name="forearm">
+</link>
+<link name="forearm">
     <xacro:LinkInertial trans="0 0 ${0.0481+(length/2)}" rpy="0 0 0" />
     <xacro:LinkVisual trans="0 0 ${0.0481+(length/2)}" rpy="0 0 0" />
     <xacro:LinkCollision trans="0 0 ${0.0481+(length/2)}" rpy="0 0 0" />
-  </link>
-  <link name="wrist_bracket">
+</link>
+<link name="wrist_bracket">
     <xacro:AxBracketInertial trans="0 0 ${0.0988+length}" rpy="1.57 0 1.57"/>
     <xacro:AxBracketVisual trans="0 0 ${0.0988+length}" rpy="1.57 0 1.57"/>
     <xacro:AxBracketCollision trans="0 0 ${0.0988+length}" rpy="1.57 0 1.57"/>
-  </link>
-  <link name="wrist_pitch_motor">
+</link>
+<link name="wrist_pitch_motor">
     <xacro:AXInertial trans="0 0 0" rpy="-1.57 0 -1.57"/>
-    <xacro:AXVisual trans="0. 0 0" rpy="-1.57 0 -1.57"/>
+    <xacro:AXVisual trans="0 0 0" rpy="-1.57 0 -1.57"/>
     <xacro:AXCollision trans="0 0 0" rpy="-1.57 0 -1.57"/>
-  </link>
-  <link name="wrist_roll_motor">
+</link>
+<link name="wrist_roll_motor">
     <xacro:AXInertial trans="0 0.015 0.0585" rpy="0 0 0"/>
     <xacro:AXVisual trans="0 0.015 0.0585" rpy="0 0 0"/>
     <xacro:AXCollision trans="0 0.015 0.0585" rpy="0 0 0"/>
-  </link>
- <link name="end_effector">
-    <xacro:BracketInertial trans="0 0 0" rpy="3.14 0 1.57"/>
-    <xacro:BracketVisual trans="0 0 0" rpy="3.14 0 -1.57"/>
-    <xacro:BracketCollision trans="0 0 0" rpy="3.14 0 1.57"/>
-  </link>
+</link>
+<link name="end_effector">
+    <xacro:F3Inertial trans="0 0 0" rpy="-1.57 3.14 1.57"/>
+    <xacro:F3Visual trans="0 0 0" rpy="-1.57 3.14 0"/>
+    <xacro:F3Collision trans="0 0 0" rpy="-1.57 3.14 1.57"/>
+</link>
+<link name="gripper_motor">
+    <xacro:AXInertial trans="0 0 0.02" rpy="0 0 0 "/>
+    <xacro:AXVisual trans="0 0 0.04" rpy="-1.57 3.14 0"/>
+    <xacro:AXCollision trans="0 0 0.02" rpy="0 0 0"/>
+</link>
+<link name="F10_bracket">
+    <xacro:F10Inertial trans="0.016 0 0.02" rpy="1.57 0 0 "/>
+    <xacro:F10Visual trans="0.016 0.02 0" rpy="0 3.14 0 "/>
+    <xacro:F10Collision trans="0.016 0 0.02" rpy="1.57 0 0 "/>
+</link>
+<link name="F9_bracket">
+    <xacro:F9Inertial trans="0.04101 0.00807 0.003" rpy="-1.57 0 -1.57"/>
+    <xacro:F9Visual trans="0.04101 0.00609 0.003" rpy="-1.57 0 -1.57 "/>
+    <xacro:F9Collision trans="0.04101 0.00807 0.003" rpy="-1.57 0 -1.57 "/>
+</link>
+<link name="F11_bracket">
+    <xacro:F11Inertial trans="0.04101 0.021785 0.003" rpy="0 -3.14 0 "/>
+    <xacro:F11Visual trans="0.04101 0.0 0.01962" rpy="-1.57 -3.14 0 "/>
+    <xacro:F11Collision trans="0.04101 0.021785 0.003" rpy="0 -3.14 0 "/>
+</link>
+<link name="F3_bracket">
+    <xacro:F3Inertial trans="-0.02 -0.01402 0" rpy="0 0 -1.57"/>
+    <xacro:F3Visual trans="-0.02 0 0.026" rpy="0 1.57 -1.57"/>
+    <xacro:F3Collision trans="-0.02 -0.01402 0" rpy="0 0 -1.57"/>
+</link>
+<link name="F6_bracket">
+    <xacro:F6Inertial trans="-0.0222 0.01304 0" rpy="0 0 -1.57"/>
+    <xacro:F6Visual trans="-0.0222 0 0.039" rpy="0 1.57 -1.57"/>
+    <xacro:F6Collision trans="-0.0222 0.01304 0" rpy="0 0 -1.57"/>
+</link>
+<link name="F11_bracket_1">
+    <xacro:F11Inertial trans="-0.026462 0.029105 0" rpy="0 0 0 "/>
+    <xacro:F11Visual trans="-0.026462 0 0.055105" rpy="1.57 0 0 "/>
+    <xacro:F11Collision trans="-0.026462 0.029105 0" rpy="0 0 0 "/>
+</link>
+<!--JOINTS-->
   <xacro:Revjoint id="shoulder_yaw" trans="0 0 0" rpy="0 0 0" parent="shoulder_yaw_motor" child="shoulder_bracket" axis="0 0 1" l="-3.14" u="3.14" v="1.0"/>
   <xacro:Revjoint id="shoulder_pitch" trans="0 0 0.0636" rpy="0 0 0" parent="shoulder_bracket" child="shoulder_pitch_motor" axis="1 0 0" l="-1.57" u="1.57" v="1.0"/>
   <xacro:FxdJoint id="s1_l2" parent="shoulder_pitch_motor" child="biscep"/>
   <xacro:FxdJoint id="l2_l2B" parent="biscep" child="elbow_bracket"/>
-  <xacro:Revjoint id="elbow" trans="0 0 ${0.0867+(length)}" rpy="0 0 0" parent="elbow_bracket" child="elbow_motor" axis="1 0 0" l="-1.57" u="1.57" v="1.0"/>
+  <xacro:Revjoint id="elbow" trans="0 0 ${0.0867+(length)}" rpy="0 0 0" parent="elbow_bracket" child="elbow_motor" axis="1 0 0" l="-1.9" u="1.85" v="1.0"/>
   <xacro:FxdJoint id="e_l3" parent="elbow_motor" child="forearm"/>
   <xacro:FxdJoint id="l3_l3B" parent="forearm" child="wrist_bracket"/>
-  <xacro:Revjoint id="wrist_pitch" trans="0 0 ${0.0988+length}" rpy="0 0 0" parent="wrist_bracket" child="wrist_pitch_motor" axis="1 0 0" l="-1.57" u="1.57" v="1.0"/>
+  <xacro:Revjoint id="wrist_pitch" trans="0 0 ${0.0988+length}" rpy="0 0 0" parent="wrist_bracket" child="wrist_pitch_motor" axis="1 0 0" l="-2.25" u="2.3" v="1.0"/>
   <xacro:FxdJoint id="WP_WR" parent="wrist_pitch_motor" child="wrist_roll_motor"/>
   <xacro:Revjoint id="wrist_roll" trans="0 0.015 0.0785" rpy="0 0 0" parent="wrist_roll_motor" child="end_effector" axis="0 0 1" l="-3.14" u="3.14" v="1.0"/>
+  <xacro:FxdJoint id="Bracket_gripper" parent="end_effector" child="gripper_motor"/>
+  <xacro:Revjoint id="gripper_joint" trans="0 0 0.04" rpy="0 0 0" parent="gripper_motor" child="F10_bracket" axis="0 1 0" l="-3.14" u="3.14" v="1.0"/>
+  <xacro:FxdJoint id="left_L" parent="F10_bracket" child="F9_bracket"/>
+  <xacro:FxdJoint id="left_H" parent="F9_bracket" child="F11_bracket"/>
+  <xacro:FxdJoint id="right_j" parent="gripper_motor" child="F3_bracket"/>
+  <xacro:FxdJoint id="right_L" parent="F3_bracket" child="F6_bracket"/>
+  <xacro:FxdJoint id="right_H" parent="F6_bracket" child="F11_bracket_1"/>
 </robot>

File: src/mobile_manipulator/model/test.urdf (robot description, URDF)
Before this commit: robot mobile_manipulator, 11 links, 10 joints
Links:
- removed link WristPitch
- removed link WristRoll
- removed link base_link
- removed link elbow
- removed link link1Bracket
- removed link link2
- removed link link2Bracket
- removed link link3
- removed link link3Bracket
- removed link shoulder1
- added link F10_bracket, mass 0.00712; collision mesh filename=package://mobile_manipulator/meshes/F10.stl scale=0.001 0.001 0.001; visual mesh filename=package://mobile_manipulator/meshes/F10.stl scale=0.001 0.001 0.001
- added link F11_bracket, mass 0.00712; collision mesh filename=package://mobile_manipulator/meshes/F11.stl scale=0.001 0.001 0.001; visual mesh filename=package://mobile_manipulator/meshes/F11.stl scale=0.001 0.001 0.001
- added link F11_bracket_1, mass 0.00712; collision mesh filename=package://mobile_manipulator/meshes/F11.stl scale=0.001 0.001 0.001; visual mesh filename=package://mobile_manipulator/meshes/F11.stl scale=0.001 0.001 0.001
- added link F3_bracket, mass 0.00712; collision mesh filename=package://mobile_manipulator/meshes/F3.stl scale=0.001 0.001 0.001; visual mesh filename=package://mobile_manipulator/meshes/F3.stl scale=0.001 0.001 0.001
- added link F6_bracket, mass 0.00712; collision mesh filename=package://mobile_manipulator/meshes/F6.stl scale=0.001 0.001 0.001; visual mesh filename=package://mobile_manipulator/meshes/F6.stl scale=0.001 0.001 0.001
- added link F9_bracket, mass 0.00712; collision mesh filename=package://mobile_manipulator/meshes/F9.stl scale=0.001 0.001 0.001; visual mesh filename=package://mobile_manipulator/meshes/F9.stl scale=0.001 0.001 0.001
- added link biscep, mass 0.00048; collision box size=0.04 0.04 0.096; visual box size=0.04 0.04 0.096
- added link elbow_bracket, mass 0.00712; collision mesh filename=package://mobile_manipulator/meshes/FR05-H101K.stl scale=0.001 0.001 0.001; visual mesh filename=package://mobile_manipulator/meshes/FR05-H101K.stl scale=0.001 0.001 0.001
- added link elbow_motor, mass 0.140; collision box size=0.041 0.0402 0.0611; visual mesh filename=package://mobile_manipulator/meshes/dynamixel_x64series.stl scale=0.001 0.001 0.001
- added link forearm, mass 0.00048; collision box size=0.04 0.04 0.096; visual box size=0.04 0.04 0.096
- added link gripper_motor, mass 0.05573; collision box size=0.032 0.04 0.05; visual mesh filename=package://mobile_manipulator/meshes/AX-12_18A - dynamixel_A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 scale=0.001 0.001 0.001
- added link shoulder_bracket, mass 0.00712; collision mesh filename=package://mobile_manipulator/meshes/FR05-H101K.stl scale=0.001 0.001 0.001; visual mesh filename=package://mobile_manipulator/meshes/FR05-H101K.stl scale=0.001 0.001 0.001
- added link shoulder_pitch_motor, mass 0.140; collision box size=0.041 0.0402 0.0611; visual mesh filename=package://mobile_manipulator/meshes/dynamixel_x64series.stl scale=0.001 0.001 0.001
- added link shoulder_yaw_motor, mass 0.140; collision box size=0.041 0.0402 0.0611; visual mesh filename=package://mobile_manipulator/meshes/dynamixel_x64series.stl scale=0.001 0.001 0.001
- added link wrist_bracket, mass 0.00712; collision mesh filename=package://mobile_manipulator/meshes/F4.stl scale=0.001 0.001 0.001; visual mesh filename=package://mobile_manipulator/meshes/F4.stl scale=0.001 0.001 0.001
- added link wrist_pitch_motor, mass 0.05573; collision box size=0.032 0.04 0.05; visual mesh filename=package://mobile_manipulator/meshes/AX-12_18A - dynamixel_A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 scale=0.001 0.001 0.001
- added link wrist_roll_motor, mass 0.05573; collision box size=0.032 0.04 0.05; visual mesh filename=package://mobile_manipulator/meshes/AX-12_18A - dynamixel_A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 scale=0.001 0.001 0.001
- link end_effector: geometry collision mesh filename=package://mobile_manipulator/meshes/F3.stl scale=0.001 0.001 0.001; visual mesh filename=package://mobile_manipulator/meshes/F3.stl scale=0.001 0.001 0.001
Joints:
- removed joint five
- removed joint four
- removed joint one
- removed joint three
- removed joint two
- added joint Bracket_gripper: type fixed, parent end_effector, child gripper_motor
- added joint elbow: type revolute, parent elbow_bracket, child elbow_motor, origin xyz=0 0 0.1827 rpy=0 0 0, axis 1 0 0, limit lower=-1.9 upper=1.85 effort=30 velocity=1.0
- added joint gripper_joint: type revolute, parent gripper_motor, child F10_bracket, origin xyz=0 0 0.04 rpy=0 0 0, axis 0 1 0, limit lower=-3.14 upper=3.14 effort=30 velocity=1.0
- added joint left_H: type fixed, parent F9_bracket, child F11_bracket
- added joint left_L: type fixed, parent F10_bracket, child F9_bracket
- added joint right_H: type fixed, parent F6_bracket, child F11_bracket_1
- added joint right_L: type fixed, parent F3_bracket, child F6_bracket
- added joint right_j: type fixed, parent gripper_motor, child F3_bracket
- added joint shoulder_pitch: type revolute, parent shoulder_bracket, child shoulder_pitch_motor, origin xyz=0 0 0.0636 rpy=0 0 0, axis 1 0 0, limit lower=-1.57 upper=1.57 effort=30 velocity=1.0
- added joint shoulder_yaw: type revolute, parent shoulder_yaw_motor, child shoulder_bracket, origin xyz=0 0 0 rpy=0 0 0, axis 0 0 1, limit lower=-3.14 upper=3.14 effort=30 velocity=1.0
- added joint wrist_pitch: type revolute, parent wrist_bracket, child wrist_pitch_motor, origin xyz=0 0 0.1948 rpy=0 0 0, axis 1 0 0, limit lower=-2.25 upper=2.3 effort=30 velocity=1.0
- added joint wrist_roll: type revolute, parent wrist_roll_motor, child end_effector, origin xyz=0 0.015 0.0785 rpy=0 0 0, axis 0 0 1, limit lower=-3.14 upper=3.14 effort=30 velocity=1.0
- joint WP_WR: child WristRoll -> wrist_roll_motor; parent WristPitch -> wrist_pitch_motor
- joint e_l3: child link3 -> forearm; parent elbow -> elbow_motor
- joint l2_l2B: child link2Bracket -> elbow_bracket; parent link2 -> biscep
- joint l3_l3B: child link3Bracket -> wrist_bracket; parent link3 -> forearm
- joint s1_l2: child link2 -> biscep; parent shoulder1 -> shoulder_pitch_motor

Commit message: Changing Link Names

File: src/mobile_manipulator/model/mobile_manipulator.xacro (robot description, xacro)
@@ -318,5 +318,5 @@
     <xacro:AXCollision trans="0 0.015 0.0585" rpy="0 0 0"/>
 </link>
-<link name="end_effector">
+<link name="wrist_roll_bracket">
     <xacro:F3Inertial trans="0 0 0" rpy="-1.57 3.14 1.57"/>
     <xacro:F3Visual trans="0 0 0" rpy="-1.57 3.14 0"/>
@@ -338,5 +338,5 @@
     <xacro:F9Collision trans="0.04101 0.00807 0.003" rpy="-1.57 0 -1.57 "/>
 </link>
-<link name="F11_bracket">
+<link name="end_effector_l">
     <xacro:F11Inertial trans="0.04101 0.021785 0.003" rpy="0 -3.14 0 "/>
     <xacro:F11Visual trans="0.04101 0.0 0.01962" rpy="-1.57 -3.14 0 "/>
@@ -353,5 +353,5 @@
     <xacro:F6Collision trans="-0.0222 0.01304 0" rpy="0 0 -1.57"/>
 </link>
-<link name="F11_bracket_1">
+<link name="end_effector_r">
     <xacro:F11Inertial trans="-0.026462 0.029105 0" rpy="0 0 0 "/>
     <xacro:F11Visual trans="-0.026462 0 0.055105" rpy="1.57 0 0 "/>
@@ -368,11 +368,11 @@
   <xacro:Revjoint id="wrist_pitch" trans="0 0 ${0.0988+length}" rpy="0 0 0" parent="wrist_bracket" child="wrist_pitch_motor" axis="1 0 0" l="-2.25" u="2.3" v="1.0"/>
   <xacro:FxdJoint id="WP_WR" parent="wrist_pitch_motor" child="wrist_roll_motor"/>
-  <xacro:Revjoint id="wrist_roll" trans="0 0.015 0.0785" rpy="0 0 0" parent="wrist_roll_motor" child="end_effector" axis="0 0 1" l="-3.14" u="3.14" v="1.0"/>
-  <xacro:FxdJoint id="Bracket_gripper" parent="end_effector" child="gripper_motor"/>
+  <xacro:Revjoint id="wrist_roll" trans="0 0.015 0.0785" rpy="0 0 0" parent="wrist_roll_motor" child="wrist_roll_bracket" axis="0 0 1" l="-3.14" u="3.14" v="1.0"/>
+  <xacro:FxdJoint id="Bracket_gripper" parent="wrist_roll_bracket" child="gripper_motor"/>
   <xacro:Revjoint id="gripper_joint" trans="0 0 0.04" rpy="0 0 0" parent="gripper_motor" child="F10_bracket" axis="0 1 0" l="-3.14" u="3.14" v="1.0"/>
   <xacro:FxdJoint id="left_L" parent="F10_bracket" child="F9_bracket"/>
-  <xacro:FxdJoint id="left_H" parent="F9_bracket" child="F11_bracket"/>
+  <xacro:FxdJoint id="left_H" parent="F9_bracket" child="end_effector_l"/>
   <xacro:FxdJoint id="right_j" parent="gripper_motor" child="F3_bracket"/>
   <xacro:FxdJoint id="right_L" parent="F3_bracket" child="F6_bracket"/>
-  <xacro:FxdJoint id="right_H" parent="F6_bracket" child="F11_bracket_1"/>
+  <xacro:FxdJoint id="right_H" parent="F6_bracket" child="end_effector_r"/>
 </robot>
