Commit message: End Effector Changed 	new file:   src/mobile_manipulator/meshes/F10.stl 	modified:   src/mobile_manipulator/model/mobile_manipulator.xacro

File: src/mobile_manipulator/model/mobile_manipulator.xacro (robot description, xacro)
@@ -146,4 +146,28 @@
     </joint>
 </xacro:macro>
+<xacro:macro name="F10Inertial" params="trans rpy">
+  <inertial>
+    <origin xyz="${trans}" rpy="${rpy}"/>
+    <mass value="0.00712" />
+    <inertia ixx="0.00000174511" iyy="0.00000379922" ixz="0.0" ixy="0.0" iyz="0.0" izz="0.00000357521" />
+  </inertial>
+</xacro:macro>
+<xacro:macro name="F10Visual" params="trans rpy">
+  <visual>
+    <origin xyz="${trans}" rpy="${rpy}"/>
+    <geometry>
+      <mesh filename="package://mobile_manipulator/meshes/F10.stl" scale="0.001 0.001 0.001" />
+    </geometry>
+    <material name="white"/>
+  </visual>
+</xacro:macro>
+<xacro:macro name="F10Collision" params="trans rpy">
+    <collision>
+      <origin xyz="${trans}" rpy="${rpy}"/>
+      <geometry>
+        <mesh filename="package://mobile_manipulator/meshes/F10.stl" scale="0.001 0.001 0.001"/>
+      </geometry>
+    </collision>
+</xacro:macro>
   <link name="shoulder_yaw_motor">
     <xacro:MXInertial trans="0 0 0" rpy="0 0 0 "/>
@@ -196,8 +220,15 @@
     <xacro:AXCollision trans="0 0.015 0.0585" rpy="0 0 0"/>
   </link>
+<!--
  <link name="end_effector">
     <xacro:BracketInertial trans="0 0 0" rpy="3.14 0 1.57"/>
     <xacro:BracketVisual trans="0 0 0" rpy="3.14 0 -1.57"/>
     <xacro:BracketCollision trans="0 0 0" rpy="3.14 0 1.57"/>
+  </link>
+   -->
+ <link name="end_effector">
+    <xacro:F10Inertial trans="0 0.015 0" rpy="1.57 0 1.57"/>
+    <xacro:F10Visual trans="0 0.015 0" rpy="1.57 0 1.57"/>
+    <xacro:F10Collision trans="0 0.015 0" rpy="1.57 0 1.57"/>
   </link>
   <xacro:Revjoint id="shoulder_yaw" trans="0 0 0" rpy="0 0 0" parent="shoulder_yaw_motor" child="shoulder_bracket" axis="0 0 1" l="-3.0357" u="3.24426" v="1.0"/>

File: src/mobile_manipulator/model/test.urdf (robot description, URDF)
Before this commit: robot mobile_manipulator, 11 links, 10 joints
Links:
- removed link WristPitch
- removed link WristRoll
- removed link base_link
- removed link elbow
- removed link link1Bracket
- removed link link2
- removed link link2Bracket
- removed link link3
- removed link link3Bracket
- removed link shoulder1
- added link biscep, mass 0.00048; collision box size=0.04 0.04 0.096; visual box size=0.04 0.04 0.096
- added link elbow_bracket, mass 0.00712; collision mesh filename=package://mobile_manipulator/meshes/FR05-H101K.stl scale=0.001 0.001 0.001; visual mesh filename=package://mobile_manipulator/meshes/FR05-H101K.stl scale=0.001 0.001 0.001
- added link elbow_motor, mass 0.140; collision box size=0.041 0.0402 0.0611; visual mesh filename=package://mobile_manipulator/meshes/dynamixel_x64series.stl scale=0.001 0.001 0.001
- added link forearm, mass 0.00048; collision box size=0.04 0.04 0.096; visual box size=0.04 0.04 0.096
- added link shoulder_bracket, mass 0.00712; collision mesh filename=package://mobile_manipulator/meshes/FR05-H101K.stl scale=0.001 0.001 0.001; visual mesh filename=package://mobile_manipulator/meshes/FR05-H101K.stl scale=0.001 0.001 0.001
- added link shoulder_pitch_motor, mass 0.140; collision box size=0.041 0.0402 0.0611; visual mesh filename=package://mobile_manipulator/meshes/dynamixel_x64series.stl scale=0.001 0.001 0.001
- added link shoulder_yaw_motor, mass 0.140; collision box size=0.041 0.0402 0.0611; visual mesh filename=package://mobile_manipulator/meshes/dynamixel_x64series.stl scale=0.001 0.001 0.001
- added link wrist_bracket, mass 0.00712; collision mesh filename=package://mobile_manipulator/meshes/F4.stl scale=0.001 0.001 0.001; visual mesh filename=package://mobile_manipulator/meshes/F4.stl scale=0.001 0.001 0.001
- added link wrist_pitch_motor, mass 0.05573; collision box size=0.032 0.04 0.05; visual mesh filename=package://mobile_manipulator/meshes/AX-12_18A - dynamixel_A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 scale=0.001 0.001 0.001
- added link wrist_roll_motor, mass 0.05573; collision box size=0.032 0.04 0.05; visual mesh filename=package://mobile_manipulator/meshes/AX-12_18A - dynamixel_A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 scale=0.001 0.001 0.001
- link end_effector: geometry collision mesh filename=package://mobile_manipulator/meshes/F10.stl scale=0.001 0.001 0.001; visual mesh filename=package://mobile_manipulator/meshes/F10.stl scale=0.001 0.001 0.001
Joints:
- removed joint five
- removed joint four
- removed joint one
- removed joint three
- removed joint two
- added joint elbow: type revolute, parent elbow_bracket, child elbow_motor, origin xyz=0 0 0.1827 rpy=0 0 0, axis 1 0 0, limit lower=-1.99 upper=1.971699219 effort=30 velocity=1.0
- added joint shoulder_pitch: type revolute, parent shoulder_bracket, child shoulder_pitch_motor, origin xyz=0 0 0.0636 rpy=0 0 0, axis 1 0 0, limit lower=-1.973232422 upper=1.916503906 effort=30 velocity=1.0
- added joint shoulder_yaw: type revolute, parent shoulder_yaw_motor, child shoulder_bracket, origin xyz=0 0 0 rpy=0 0 0, axis 0 0 1, limit lower=-3.0357 upper=3.24426 effort=30 velocity=1.0
- added joint wrist_pitch: type revolute, parent wrist_bracket, child wrist_pitch_motor, origin xyz=0 0 0.1948 rpy=0 0 0, axis 1 0 0, limit lower=-2.36344086 upper=2.368556533 effort=30 velocity=1.0
- added joint wrist_roll: type revolute, parent wrist_roll_motor, child end_effector, origin xyz=0 0.015 0.0785 rpy=0 0 0, axis 0 0 1, limit lower=-3.14 upper=+3.14 effort=30 velocity=1.0
- joint WP_WR: child WristRoll -> wrist_roll_motor; parent WristPitch -> wrist_pitch_motor
- joint e_l3: child link3 -> forearm; parent elbow -> elbow_motor
- joint l2_l2B: child link2Bracket -> elbow_bracket; parent link2 -> biscep
- joint l3_l3B: child link3Bracket -> wrist_bracket; parent link3 -> forearm
- joint s1_l2: child link2 -> biscep; parent shoulder1 -> shoulder_pitch_motor

Commit message: Toll Roll Motor Orientation Changed

File: src/mobile_manipulator/model/mobile_manipulator.xacro (robot description, xacro)
@@ -11,4 +11,5 @@
 <xacro:property name="AXDepth" value="0.04"/>
 <xacro:property name="length" value="0.096"/>
+<!-- MACROS -->
 <xacro:macro name="MXInertial" params="trans rpy">
   <inertial>
@@ -170,4 +171,5 @@
     </collision>
 </xacro:macro>
+<!-- LINKS -->
   <link name="shoulder_yaw_motor">
     <xacro:MXInertial trans="0 0 0" rpy="0 0 0 "/>
@@ -216,8 +218,8 @@
   </link>
   <link name="wrist_roll_motor">
-    <xacro:AXInertial trans="0 0.015 0.0585" rpy="0 0 0"/>
-    <xacro:AXVisual trans="0 0.015 0.0585" rpy="0 0 0"/>
-    <xacro:AXCollision trans="0 0.015 0.0585" rpy="0 0 0"/>
-  </link>
+    <xacro:AXInertial trans="0 0.035 0.027" rpy="-1.57 3.14 0"/>
+    <xacro:AXVisual trans="0 0.035 0.027" rpy="-1.57 3.14 0"/>
+    <xacro:AXCollision trans="0 0.035 0.027" rpy="-1.57 3.14 0"/>
+  </link> <!--trans="0 0.015 0.0585" rpy="-1.57 0 0"-->
 <!--
  <link name="end_effector">
@@ -228,8 +230,9 @@
    -->
  <link name="end_effector">
-    <xacro:F10Inertial trans="0 0.015 0" rpy="1.57 0 1.57"/>
-    <xacro:F10Visual trans="0 0.015 0" rpy="1.57 0 1.57"/>
-    <xacro:F10Collision trans="0 0.015 0" rpy="1.57 0 1.57"/>
-  </link>
+    <xacro:F10Inertial trans="0 0.040 -0.016" rpy="1.57 1.57 1.57"/>
+    <xacro:F10Visual trans="0 0.040 -0.016" rpy="1.57 1.57 1.57"/>
+    <xacro:F10Collision trans="0 0.040 -0.016" rpy="1.57 1.57 1.57"/>
+  </link><!--trans="0 0.015 0" rpy="1.57 0 1.57"-->
+ <!-- JOINTS -->
   <xacro:Revjoint id="shoulder_yaw" trans="0 0 0" rpy="0 0 0" parent="shoulder_yaw_motor" child="shoulder_bracket" axis="0 0 1" l="-3.0357" u="3.24426" v="1.0"/>
   <xacro:Revjoint id="shoulder_pitch" trans="0 0 0.0636" rpy="0 0 0" parent="shoulder_bracket" child="shoulder_pitch_motor" axis="1 0 0" l="-1.973232422" u="1.916503906" v="1.0"/>
@@ -241,5 +244,5 @@
   <xacro:Revjoint id="wrist_pitch" trans="0 0 ${0.0988+length}" rpy="0 0 0" parent="wrist_bracket" child="wrist_pitch_motor" axis="1 0 0" l="-2.36344086" u="2.368556533" v="1.0"/>
   <xacro:FxdJoint id="WP_WR" parent="wrist_pitch_motor" child="wrist_roll_motor"/>
-  <xacro:Revjoint id="wrist_roll" trans="0 0.015 0.0785" rpy="0 0 0" parent="wrist_roll_motor" child="end_effector" axis="0 0 1" l="-3.14" u="+3.14" v="1.0"/>
+  <xacro:Revjoint id="wrist_roll" trans="0 0.015 0.027" rpy="0 0 0" parent="wrist_roll_motor" child="end_effector" axis="0 1 0" l="-3.14" u="+3.14" v="1.0"/>
   <!-- <xacro:Revjoint id="wrist_roll" trans="0 0.015 0.0785" rpy="0 0 0" parent="wrist_roll_motor" child="end_effector" axis="0 0 1" l="-2.616666666" u="2.616666666" v="1.0"/> -->
 </robot>

File: src/mobile_manipulator/model/test.urdf (robot description, URDF)
Before this commit: robot mobile_manipulator, 11 links, 10 joints
Joints:
- joint wrist_roll: axis 0 0 1 -> 0 1 0; origin xyz=0 0.015 0.0785 rpy=0 0 0 -> xyz=0 0.015 0.027 rpy=0 0 0

Commit message: Roll motor shifted

File: src/mobile_manipulator/model/mobile_manipulator.xacro (robot description, xacro)
@@ -219,7 +219,7 @@
   <link name="wrist_roll_motor">
     <xacro:AXInertial trans="0 0.035 0.027" rpy="-1.57 3.14 0"/>
-    <xacro:AXVisual trans="0 0.035 0.027" rpy="-1.57 3.14 0"/>
+    <xacro:AXVisual trans="0 0 0.075" rpy="-1.57 3.14 0"/>
     <xacro:AXCollision trans="0 0.035 0.027" rpy="-1.57 3.14 0"/>
-  </link> <!--trans="0 0.015 0.0585" rpy="-1.57 0 0"-->
+  </link> <!--trans="0 0.015 0.0585" trans1="0 0.035 0.027" rpy="-1.57 0 0"-->
 <!--
  <link name="end_effector">
@@ -231,5 +231,5 @@
  <link name="end_effector">
     <xacro:F10Inertial trans="0 0.040 -0.016" rpy="1.57 1.57 1.57"/>
-    <xacro:F10Visual trans="0 0.040 -0.016" rpy="1.57 1.57 1.57"/>
+    <xacro:F10Visual trans="0 0.005 -0.016" rpy="1.57 1.57 1.57"/>
     <xacro:F10Collision trans="0 0.040 -0.016" rpy="1.57 1.57 1.57"/>
   </link><!--trans="0 0.015 0" rpy="1.57 0 1.57"-->
@@ -244,5 +244,5 @@
   <xacro:Revjoint id="wrist_pitch" trans="0 0 ${0.0988+length}" rpy="0 0 0" parent="wrist_bracket" child="wrist_pitch_motor" axis="1 0 0" l="-2.36344086" u="2.368556533" v="1.0"/>
   <xacro:FxdJoint id="WP_WR" parent="wrist_pitch_motor" child="wrist_roll_motor"/>
-  <xacro:Revjoint id="wrist_roll" trans="0 0.015 0.027" rpy="0 0 0" parent="wrist_roll_motor" child="end_effector" axis="0 1 0" l="-3.14" u="+3.14" v="1.0"/>
+  <xacro:Revjoint id="wrist_roll" trans="0 0.015 0.077" rpy="0 3.14 0" parent="wrist_roll_motor" child="end_effector" axis="0 1 0" l="-3.14" u="+3.14" v="1.0"/>
   <!-- <xacro:Revjoint id="wrist_roll" trans="0 0.015 0.0785" rpy="0 0 0" parent="wrist_roll_motor" child="end_effector" axis="0 0 1" l="-2.616666666" u="2.616666666" v="1.0"/> -->
 </robot>

File: src/mobile_manipulator/model/test.urdf (robot description, URDF)
Before this commit: robot mobile_manipulator, 11 links, 10 joints
Joints:
- joint wrist_roll: origin xyz=0 0.015 0.027 rpy=0 0 0 -> xyz=0 0.015 0.077 rpy=0 3.14 0

Commit message: Added gripper to new URDF
	modified:   mobile_manipulator.xacro
	new file:   testing.urdf

File: src/mobile_manipulator/model/mobile_manipulator.xacro (robot description, xacro)
@@ -222,16 +222,15 @@
     <xacro:AXCollision trans="0 0.035 0.027" rpy="-1.57 3.14 0"/>
   </link> <!--trans="0 0.015 0.0585" trans1="0 0.035 0.027" rpy="-1.57 0 0"-->
-<!--
- <link name="end_effector">
-    <xacro:BracketInertial trans="0 0 0" rpy="3.14 0 1.57"/>
-    <xacro:BracketVisual trans="0 0 0" rpy="3.14 0 -1.57"/>
-    <xacro:BracketCollision trans="0 0 0" rpy="3.14 0 1.57"/>
-  </link>
-   -->
- <link name="end_effector">
+  <link name="gripper_motor">
+    <xacro:AXInertial trans="0.03 0.037 0" rpy="-1.57 3.14 0"/>
+    <xacro:AXVisual trans="0 0.037 0" rpy="0 -1.57 0"/>
+    <xacro:AXCollision trans="0 0.035 0.027" rpy="-1.57 3.14 0"/>
+  </link>
+ <!-- <link name="end_effector">
     <xacro:F10Inertial trans="0 0.040 -0.016" rpy="1.57 1.57 1.57"/>
     <xacro:F10Visual trans="0 0.005 -0.016" rpy="1.57 1.57 1.57"/>
     <xacro:F10Collision trans="0 0.040 -0.016" rpy="1.57 1.57 1.57"/>
-  </link><!--trans="0 0.015 0" rpy="1.57 0 1.57"-->
+  </link> -->
+  <!-- trans="0 0.015 0" rpy="1.57 0 1.57" -->
  <!-- JOINTS -->
   <xacro:Revjoint id="shoulder_yaw" trans="0 0 0" rpy="0 0 0" parent="shoulder_yaw_motor" child="shoulder_bracket" axis="0 0 1" l="-3.0357" u="3.24426" v="1.0"/>
@@ -244,5 +243,6 @@
   <xacro:Revjoint id="wrist_pitch" trans="0 0 ${0.0988+length}" rpy="0 0 0" parent="wrist_bracket" child="wrist_pitch_motor" axis="1 0 0" l="-2.36344086" u="2.368556533" v="1.0"/>
   <xacro:FxdJoint id="WP_WR" parent="wrist_pitch_motor" child="wrist_roll_motor"/>
-  <xacro:Revjoint id="wrist_roll" trans="0 0.015 0.077" rpy="0 3.14 0" parent="wrist_roll_motor" child="end_effector" axis="0 1 0" l="-3.14" u="+3.14" v="1.0"/>
+  <!-- <xacro:Revjoint id="wrist_roll" trans="0 0.015 0.077" rpy="0 3.14 0" parent="wrist_roll_motor" child="end_effector" axis="0 1 0" l="-3.14" u="+3.14" v="1.0"/> -->
+  <xacro:Revjoint id="wrist_roll" trans="0.041 0.02 0.021" rpy="0 3.14 0" parent="wrist_roll_motor" child="gripper_motor" axis="0 1 0" l="-3.14" u="+3.14" v="1.0"/>
   <!-- <xacro:Revjoint id="wrist_roll" trans="0 0.015 0.0785" rpy="0 0 0" parent="wrist_roll_motor" child="end_effector" axis="0 0 1" l="-2.616666666" u="2.616666666" v="1.0"/> -->
 </robot>

Commit message: Almost done with the new XACRO, added j plate, end effector pending
	new file:   ../meshes/base_dyna.stl
	new file:   ../meshes/base_und.stl
	new file:   ../meshes/gripper_Centering.pdf
	new file:   ../meshes/gripper_Centering.stl
	modified:   mobile_manipulator.xacro

File: src/mobile_manipulator/model/mobile_manipulator.xacro (robot description, xacro)
@@ -132,4 +132,29 @@
     </collision>
 </xacro:macro>
+<!-- Macros of the J plate -->
+<xacro:macro name="roll_j_plate_Inertial" params="trans rpy">
+  <inertial>
+    <origin xyz="${trans}" rpy="${rpy}" />
+    <mass value="0.140" />
+    <inertia ixx="0.000050799110" ixy="0.0" ixz="0.0" iyy="0.00002857215" iyz="0.00000051457" izz="0.000043394" />
+  </inertial>
+</xacro:macro>
+<xacro:macro name="roll_j_plate_Visual" params="trans rpy">
+  <visual>
+    <origin xyz="${trans}" rpy="${rpy}"/>
+    <geometry>
+      <mesh filename="package://mobile_manipulator/meshes/gripper_Centering.stl" scale="0.001 0.001 0.001"/>
+    </geometry>
+    <material name="white"/>
+  </visual>
+</xacro:macro>
+<xacro:macro name="roll_j_plate_Collision" params="trans rpy">
+    <collision>
+      <origin xyz="${trans}" rpy="${rpy}"/>
+      <geometry>
+        <mesh filename="package://mobile_manipulator/meshes/gripper_Centering.stl" scale="0.001 0.001 0.001"/>
+      </geometry>
+    </collision>
+</xacro:macro>
 <xacro:macro name="Revjoint" params="id trans rpy parent child axis l u v">
     <joint name="${id}" type="revolute">
@@ -179,5 +204,5 @@
   <link name="shoulder_bracket">
     <xacro:BracketInertial trans="0 0 0.025" rpy="0 3.14 0 "/>
-    <xacro:BracketVisual trans="0 0 0.025" rpy="0 3.14 0 "/>
+    <xacro:BracketVisual trans="0 0 0.0" rpy="0 3.14 0 "/>
     <xacro:BracketCollision trans="0 0 0.025" rpy="0 3.14 0 "/>
   </link>
@@ -188,12 +213,12 @@
   </link>
   <link name="biscep">
-    <xacro:LinkInertial trans="0 0 ${0.0481+(length/2)}" rpy="0 0 0" />
-    <xacro:LinkVisual trans="0 0 ${0.0481+(length/2)}" rpy="0 0 0" />
-    <xacro:LinkCollision trans="0 0 ${0.0481+(length/2)}" rpy="0 0 0" />
+    <xacro:LinkInertial trans="0 0 ${0.051+(length/2)}" rpy="0 0 0" />
+    <xacro:LinkVisual trans="0 0 ${0.051+(length/2)}" rpy="0 0 0" />
+    <xacro:LinkCollision trans="0 0 ${0.051+(length/2)}" rpy="0 0 0" />
   </link>
   <link name="elbow_bracket">
-    <xacro:BracketInertial trans="0 0 ${0.0481+length}" rpy="0 3.14 0"/>
-    <xacro:BracketVisual trans="0 0 ${0.0481+length}" rpy="0 3.14 0"/>
-    <xacro:BracketCollision trans="0 0 ${0.0481+length}" rpy="0 3.14 0"/>
+    <xacro:BracketInertial trans="0 0 ${0.052+length}" rpy="0 3.14 0"/>
+    <xacro:BracketVisual trans="0 0 ${0.052+length}" rpy="0 3.14 0"/>
+    <xacro:BracketCollision trans="0 0 ${0.052+length}" rpy="0 3.14 0"/>
   </link>
   <link name="elbow_motor">
@@ -203,26 +228,31 @@
   </link>
   <link name="forearm">
-    <xacro:LinkInertial trans="0 0 ${0.0481+(length/2)}" rpy="0 0 0" />
-    <xacro:LinkVisual trans="0 0 ${0.0481+(length/2)}" rpy="0 0 0" />
-    <xacro:LinkCollision trans="0 0 ${0.0481+(length/2)}" rpy="0 0 0" />
+    <xacro:LinkInertial trans="0 0 ${0.052+(length/2)}" rpy="0 0 0" />
+    <xacro:LinkVisual trans="0 0 ${0.052+(length/2)}" rpy="0 0 0" />
+    <xacro:LinkCollision trans="0 0 ${0.052+(length/2)}" rpy="0 0 0" />
   </link>
   <link name="wrist_bracket">
-    <xacro:AxBracketInertial trans="0 0 ${0.0988+length}" rpy="1.57 0 1.57"/>
-    <xacro:AxBracketVisual trans="0 0 ${0.0988+length}" rpy="1.57 0 1.57"/>
-    <xacro:AxBracketCollision trans="0 0 ${0.0988+length}" rpy="1.57 0 1.57"/>
+    <xacro:AxBracketInertial trans="0 0 ${0.052+length+0.054}" rpy="1.57 0 1.57"/>
+    <xacro:AxBracketVisual trans="0 0 ${0.052+length+0.054}" rpy="1.57 0 1.57"/>
+    <xacro:AxBracketCollision trans="0 0 ${0.052+length+0.054}" rpy="1.57 0 1.57"/>
   </link>
   <link name="wrist_pitch_motor">
     <xacro:AXInertial trans="0 0 0" rpy="-1.57 0 -1.57"/>
-    <xacro:AXVisual trans="0. 0 0" rpy="-1.57 0 -1.57"/>
+    <xacro:AXVisual trans="0 0 0" rpy="-1.57 0 -1.57"/>
     <xacro:AXCollision trans="0 0 0" rpy="-1.57 0 -1.57"/>
   </link>
   <link name="wrist_roll_motor">
-    <xacro:AXInertial trans="0 0.035 0.027" rpy="-1.57 3.14 0"/>
-    <xacro:AXVisual trans="0 0 0.075" rpy="-1.57 3.14 0"/>
-    <xacro:AXCollision trans="0 0.035 0.027" rpy="-1.57 3.14 0"/>
+    <xacro:AXInertial trans="0 0 0.078" rpy="-1.57 3.14 0"/>
+    <xacro:AXVisual trans="0 0 0.078" rpy="-1.57 3.14 0"/>
+    <xacro:AXCollision trans="0 0 0.078" rpy="-1.57 3.14 0"/>
   </link> <!--trans="0 0.015 0.0585" trans1="0 0.035 0.027" rpy="-1.57 0 0"-->
-  <link name="gripper_motor">
+  <link name="roll_j_plate">
+    <xacro:roll_j_plate_Inertial trans="0 0 0" rpy="0 0 0"/>
+    <xacro:roll_j_plate_Visual trans="0 0.053 -0.025" rpy="1.57 0 -1.57"/>
+    <xacro:roll_j_plate_Collision trans="0 0 0" rpy="0 0 0"/>
+  </link>
+<link name="gripper_motor">
     <xacro:AXInertial trans="0.03 0.037 0" rpy="-1.57 3.14 0"/>
-    <xacro:AXVisual trans="0 0.037 0" rpy="0 -1.57 0"/>
+    <xacro:AXVisual trans="0 0.053 0" rpy="0 -1.57 1.57"/>
     <xacro:AXCollision trans="0 0.035 0.027" rpy="-1.57 3.14 0"/>
   </link>
@@ -234,15 +264,16 @@
   <!-- trans="0 0.015 0" rpy="1.57 0 1.57" -->
  <!-- JOINTS -->
-  <xacro:Revjoint id="shoulder_yaw" trans="0 0 0" rpy="0 0 0" parent="shoulder_yaw_motor" child="shoulder_bracket" axis="0 0 1" l="-3.0357" u="3.24426" v="1.0"/>
-  <xacro:Revjoint id="shoulder_pitch" trans="0 0 0.0636" rpy="0 0 0" parent="shoulder_bracket" child="shoulder_pitch_motor" axis="1 0 0" l="-1.973232422" u="1.916503906" v="1.0"/>
+  <xacro:Revjoint id="shoulder_yaw" trans="0 0 0.025" rpy="0 0 0" parent="shoulder_yaw_motor" child="shoulder_bracket" axis="0 0 1" l="-3.0357" u="3.24426" v="1.0"/>
+  <xacro:Revjoint id="shoulder_pitch" trans="0 0 0.035" rpy="0 0 0" parent="shoulder_bracket" child="shoulder_pitch_motor" axis="1 0 0" l="-1.973232422" u="1.916503906" v="1.0"/>
   <xacro:FxdJoint id="s1_l2" parent="shoulder_pitch_motor" child="biscep"/>
   <xacro:FxdJoint id="l2_l2B" parent="biscep" child="elbow_bracket"/>
-  <xacro:Revjoint id="elbow" trans="0 0 ${0.0867+(length)}" rpy="0 0 0" parent="elbow_bracket" child="elbow_motor" axis="1 0 0" l="-1.99" u="1.971699219" v="1.0"/>
+  <xacro:Revjoint id="elbow" trans="0 0 ${0.052 + (length) + 0.038}" rpy="0 0 0" parent="elbow_bracket" child="elbow_motor" axis="1 0 0" l="-1.99" u="1.971699219" v="1.0"/>
   <xacro:FxdJoint id="e_l3" parent="elbow_motor" child="forearm"/>
   <xacro:FxdJoint id="l3_l3B" parent="forearm" child="wrist_bracket"/>
-  <xacro:Revjoint id="wrist_pitch" trans="0 0 ${0.0988+length}" rpy="0 0 0" parent="wrist_bracket" child="wrist_pitch_motor" axis="1 0 0" l="-2.36344086" u="2.368556533" v="1.0"/>
-  <xacro:FxdJoint id="WP_WR" parent="wrist_pitch_motor" child="wrist_roll_motor"/>
-  <!-- <xacro:Revjoint id="wrist_roll" trans="0 0.015 0.077" rpy="0 3.14 0" parent="wrist_roll_motor" child="end_effector" axis="0 1 0" l="-3.14" u="+3.14" v="1.0"/> -->
-  <xacro:Revjoint id="wrist_roll" trans="0.041 0.02 0.021" rpy="0 3.14 0" parent="wrist_roll_motor" child="gripper_motor" axis="0 1 0" l="-3.14" u="+3.14" v="1.0"/>
-  <!-- <xacro:Revjoint id="wrist_roll" trans="0 0.015 0.0785" rpy="0 0 0" parent="wrist_roll_motor" child="end_effector" axis="0 0 1" l="-2.616666666" u="2.616666666" v="1.0"/> -->
+  <xacro:Revjoint id="wrist_pitch" trans="0 0 ${length + 0.052 + 0.054}" rpy="0 0 0" parent="wrist_bracket" child="wrist_pitch_motor" axis="1 0 0" l="-2.36344086" u="2.368556533" v="1.0"/>
+  <xacro:FxdJoint id="WP_WR" parent="wrist_pitch_motor" child="wrist_roll_motor" />
+  <!-- <xacro:Revjoint id="wrist_roll" trans="0 0 0.078" rpy="0 0 -1.57" parent="wrist_roll_motor" child="gripper_motor" axis="0 1 0" l="-3.14" u="+3.14" v="1.0"/> -->
+  <xacro:Revjoint id="wrist_roll" trans="0 0.02 0.082" rpy="0 0 -1.57" parent="wrist_roll_motor" child="roll_j_plate" axis="1 0 0" l="-3.14" u="+3.14" v="1.0"/>
+  <xacro:FxdJoint id="end_effector" parent="roll_j_plate" child="gripper_motor" />
+  <!-- <xacro:FxdJoint id="roll_plate" parent="gripper_motor" child="" />  -->
 </robot>

File: src/mobile_manipulator/model/testing.urdf (robot description, URDF)
Before this commit: robot mobile_manipulator, 11 links, 10 joints
Links:
- added link roll_j_plate, mass 0.140; collision mesh filename=package://mobile_manipulator/meshes/gripper_Centering.stl scale=0.001 0.001 0.001; visual mesh filename=package://mobile_manipulator/meshes/gripper_Centering.stl scale=0.001 0.001 0.001
Joints:
- added joint end_effector: type fixed, parent roll_j_plate, child gripper_motor
- joint elbow: origin xyz=0 0 0.1827 rpy=0 0 0 -> xyz=0 0 0.186 rpy=0 0 0
- joint shoulder_pitch: origin xyz=0 0 0.0636 rpy=0 0 0 -> xyz=0 0 0.035 rpy=0 0 0
- joint shoulder_yaw: origin xyz=0 0 0 rpy=0 0 0 -> xyz=0 0 0.025 rpy=0 0 0
- joint wrist_pitch: origin xyz=0 0 0.1948 rpy=0 0 0 -> xyz=0 0 0.202 rpy=0 0 0
- joint wrist_roll: axis 0 1 0 -> 1 0 0; child gripper_motor -> roll_j_plate; origin xyz=0.041 0.02 0.021 rpy=0 3.14 0 -> xyz=0 0.02 0.082 rpy=0 0 -1.57
