Commit message: New xacro complete with under actuated gripper by two man team Added the gripper motor to tilt.yaml and controller_manager Tried moving the gripper motor with tilt_controller launch file publishing to the topic
	modified:   src/mobile_manipulator/model/mobile_manipulator.xacro
	modified:   src/mobile_manipulator/model/testing.urdf
	modified:   src/my_dynamixel_tutorial/launch/controller_manager.launch
	renamed:    src/my_dynamixel_tutorial/launch/_start_tilt_controller.launch -> src/my_dynamixel_tutorial/launch/start_tilt_controller.launch
	modified:   src/my_dynamixel_tutorial/scripts/state_publisher.py
	modified:   src/my_dynamixel_tutorial/tilt.yaml

File: src/mobile_manipulator/model/mobile_manipulator.xacro (robot description, xacro)
@@ -157,4 +157,29 @@
     </collision>
 </xacro:macro>
+<!-- Macros of the gripper -->
+<xacro:macro name="gripper_Inertial" params="trans rpy">
+  <inertial>
+    <origin xyz="${trans}" rpy="${rpy}" />
+    <mass value="0.140" />
+    <inertia ixx="0.000050799110" ixy="0.0" ixz="0.0" iyy="0.00002857215" iyz="0.00000051457" izz="0.000043394" />
+  </inertial>
+</xacro:macro>
+<xacro:macro name="gripper_Visual" params="trans rpy">
+  <visual>
+    <origin xyz="${trans}" rpy="${rpy}"/>
+    <geometry>
+      <mesh filename="package://mobile_manipulator/meshes/gripper.stl" scale="0.001 0.001 0.001"/>
+    </geometry>
+    <material name="white"/>
+  </visual>
+</xacro:macro>
+<xacro:macro name="gripper_Collision" params="trans rpy">
+    <collision>
+      <origin xyz="${trans}" rpy="${rpy}"/>
+      <geometry>
+        <mesh filename="package://mobile_manipulator/meshes/gripper.stl" scale="0.001 0.001 0.001"/>
+      </geometry>
+    </collision>
+</xacro:macro>
 <xacro:macro name="Revjoint" params="id trans rpy parent child axis l u v">
     <joint name="${id}" type="revolute">
@@ -246,5 +271,5 @@
     <xacro:AXVisual trans="0 0 0.078" rpy="-1.57 3.14 0"/>
     <xacro:AXCollision trans="0 0 0.078" rpy="-1.57 3.14 0"/>
-  </link> <!--trans="0 0.015 0.0585" trans1="0 0.035 0.027" rpy="-1.57 0 0"-->
+  </link>
   <link name="roll_j_plate">
     <xacro:roll_j_plate_Inertial trans="0 0 0" rpy="0 0 0"/>
@@ -252,15 +277,9 @@
     <xacro:roll_j_plate_Collision trans="0 0 0" rpy="0 0 0"/>
   </link>
-<link name="gripper_motor">
-    <xacro:AXInertial trans="0.03 0.037 0" rpy="-1.57 3.14 0"/>
-    <xacro:AXVisual trans="0 -0.041 0.021" rpy="0 0 1.57"/>
-    <xacro:AXCollision trans="0 0.035 0.027" rpy="-1.57 3.14 0"/>
-  </link>
- <!-- <link name="end_effector">
-    <xacro:F10Inertial trans="0 0.040 -0.016" rpy="1.57 1.57 1.57"/>
-    <xacro:F10Visual trans="0 0.005 -0.016" rpy="1.57 1.57 1.57"/>
-    <xacro:F10Collision trans="0 0.040 -0.016" rpy="1.57 1.57 1.57"/>
-  </link> -->
-  <!-- trans="0 0.015 0" rpy="1.57 0 1.57" -->
+ <link name="gripper">
+    <xacro:gripper_Inertial trans="0 0 0" rpy="0 0 0"/>
+    <xacro:gripper_Visual trans="-0.069 -0.016 0.004" rpy="0 0 1.57"/>
+    <xacro:gripper_Collision trans="0 0 0" rpy="0 0 0"/>
+  </link>
  <!-- JOINTS -->
   <xacro:Revjoint id="shoulder_yaw" trans="0 0 0.025" rpy="0 0 0" parent="shoulder_yaw_motor" child="shoulder_bracket" axis="0 0 1" l="-3.0357" u="3.24426" v="1.0"/>
@@ -273,7 +292,5 @@
   <xacro:Revjoint id="wrist_pitch" trans="0 0 ${length + 0.052 + 0.054}" rpy="0 0 0" parent="wrist_bracket" child="wrist_pitch_motor" axis="1 0 0" l="-2.36344086" u="2.368556533" v="1.0"/>
   <xacro:FxdJoint id="WP_WR" parent="wrist_pitch_motor" child="wrist_roll_motor" />
-  <!-- <xacro:Revjoint id="wrist_roll" trans="0 0 0.078" rpy="0 0 -1.57" parent="wrist_roll_motor" child="gripper_motor" axis="0 1 0" l="-3.14" u="+3.14" v="1.0"/> -->
   <xacro:Revjoint id="wrist_roll" trans="0 0.02 0.082" rpy="0 0 -1.57" parent="wrist_roll_motor" child="roll_j_plate" axis="1 0 0" l="-3.14" u="+3.14" v="1.0"/>
-  <xacro:FxdJoint id="end_effector" parent="roll_j_plate" child="gripper_motor" />
-  <!-- <xacro:FxdJoint id="roll_plate" parent="gripper_motor" child="" />  -->
+  <xacro:FxdJoint id="roll_plate_gripper" parent="roll_j_plate" child="gripper" />
 </robot>

File: src/mobile_manipulator/model/testing.urdf (robot description, URDF)
Before this commit: robot mobile_manipulator, 12 links, 11 joints
Links:
- removed link gripper_motor
- added link gripper, mass 0.140; collision mesh filename=package://mobile_manipulator/meshes/gripper.stl scale=0.001 0.001 0.001; visual mesh filename=package://mobile_manipulator/meshes/gripper.stl scale=0.001 0.001 0.001
Joints:
- removed joint end_effector
- added joint roll_plate_gripper: type fixed, parent roll_j_plate, child gripper
