Commit message: IKFast Finally Working **TODO: Try to change IKFast code to implement our IK solver
		new folder:   logs/*
The Equations	new file:   src/mobile_manipulator/model/ikfast61_arm.cpp
	modified:   src/mobile_manipulator/model/mobile_manipulator.dae
	modified:   src/mobile_manipulator/model/mobile_manipulator.urdf
**		new folder:   src/mobile_manipulator_ikfast_arm_plugin/*
**		modified:   src/mobile_manipulator_moveit_config/config/kinematics.yaml

File: src/mobile_manipulator/model/mobile_manipulator.urdf (robot description, URDF)
Before this commit: robot mobile_manipulator, 11 links, 10 joints
Links:
- link end_effector: geometry collision mesh filename=package://mobile_manipulator/meshes/F10.stl scale=0.001 0.001 0.001; visual mesh filename=package://mobile_manipulator/meshes/F10.stl scale=0.001 0.001 0.001
Joints:
- joint wrist_roll: axis 0 0 1 -> 0 1 0; limit lower=-2.616666666 upper=2.616666666 effort=30 velocity=1.0 -> lower=-3.14 upper=+3.14 effort=30 velocity=1.0; origin xyz=0 0.015 0.0785 rpy=0 0 0 -> xyz=0 0.015 0.027 rpy=0 0 0

Commit message: IKFast now working, the arm can now move in the x direction
	modified:   src/move_group/scripts/inverse_kinematics.py
	modified:   src/move_group/scripts/library_compute_cartesian_path.py

File: src/mobile_manipulator/model/mobile_manipulator.urdf (robot description, URDF)
Before this commit: robot mobile_manipulator, 11 links, 10 joints
Joints:
- joint wrist_roll: origin xyz=0 0.015 0.027 rpy=0 0 0 -> xyz=0 0.015 0.077 rpy=0 3.14 0

Commit message: Final Urdf and xacro done

File: src/mobile_manipulator/model/mobile_manipulator.urdf (robot description, URDF)
Before this commit: robot mobile_manipulator, 11 links, 10 joints
Links:
- removed link end_effector
- added link gripper, mass 0.140; collision mesh filename=package://mobile_manipulator/meshes/gripper.stl scale=0.001 0.001 0.001; visual mesh filename=package://mobile_manipulator/meshes/gripper.stl scale=0.001 0.001 0.001
- added link roll_j_plate, mass 0.140; collision mesh filename=package://mobile_manipulator/meshes/gripper_Centering.stl scale=0.001 0.001 0.001; visual mesh filename=package://mobile_manipulator/meshes/gripper_Centering.stl scale=0.001 0.001 0.001
Joints:
- added joint roll_plate_gripper: type fixed, parent roll_j_plate, child gripper
- joint elbow: origin xyz=0 0 0.1827 rpy=0 0 0 -> xyz=0 0 0.186 rpy=0 0 0
- joint shoulder_pitch: origin xyz=0 0 0.0636 rpy=0 0 0 -> xyz=0 0 0.035 rpy=0 0 0
- joint shoulder_yaw: origin xyz=0 0 0 rpy=0 0 0 -> xyz=0 0 0.025 rpy=0 0 0
- joint wrist_pitch: origin xyz=0 0 0.1948 rpy=0 0 0 -> xyz=0 0 0.202 rpy=0 0 0
- joint wrist_roll: axis 0 1 0 -> 1 0 0; child end_effector -> roll_j_plate; origin xyz=0 0.015 0.077 rpy=0 3.14 0 -> xyz=0 0.02 0.082 rpy=0 0 -1.57

File: src/mobile_manipulator/model/mobile_manipulator.xacro (robot description, xacro)
@@ -229,6 +229,6 @@
   <link name="shoulder_bracket">
     <xacro:BracketInertial trans="0 0 0.025" rpy="0 3.14 0 "/>
-    <xacro:BracketVisual trans="0 0 0.0" rpy="0 3.14 0 "/>
-    <xacro:BracketCollision trans="0 0 0.025" rpy="0 3.14 0 "/>
+    <xacro:BracketVisual trans="0 0 0" rpy="0 3.14 0 "/>
+    <xacro:BracketCollision trans="0 0 0" rpy="0 3.14 0 "/>
   </link>
   <link name="shoulder_pitch_motor">
@@ -250,5 +250,5 @@
     <xacro:MXInertial trans="0 0 0" rpy="1.57 0 0"/>
     <xacro:MXVisual trans="0 0 0" rpy="1.57 3.14 -1.57"/>
-    <xacro:MXCollision trans="0 0 0" rpy="1.57 0 0"/>
+    <xacro:MXCollision trans="0 0 0" rpy="1.57 3.14 -1.57"/>
   </link>
   <link name="forearm">
@@ -275,10 +275,10 @@
     <xacro:roll_j_plate_Inertial trans="0 0 0" rpy="0 0 0"/>
     <xacro:roll_j_plate_Visual trans="0 0.021 0.048" rpy="0 1.57 3.14"/>
-    <xacro:roll_j_plate_Collision trans="0 0 0" rpy="0 0 0"/>
+    <xacro:roll_j_plate_Collision trans="0 0.021 0.048" rpy="0 1.57 3.14"/>
   </link>
  <link name="gripper">
     <xacro:gripper_Inertial trans="0 0 0" rpy="0 0 0"/>
     <xacro:gripper_Visual trans="-0.069 -0.016 0.004" rpy="0 0 1.57"/>
-    <xacro:gripper_Collision trans="0 0 0" rpy="0 0 0"/>
+    <xacro:gripper_Collision trans="-0.069 -0.016 0.004" rpy="0 0 1.57"/>
   </link>
  <!-- JOINTS -->

Commit message: Ran the setup_assistant on the new URDF file Tried generating the ikfast plugin but couldnt run start.launch, it says failed to load plugin

File: src/mobile_manipulator/model/mobile_manipulator.urdf (robot description, URDF)
Before this commit: robot mobile_manipulator, 12 links, 11 joints
Joints:
- joint wrist_roll: limit lower=-3.14 upper=+3.14 effort=30 velocity=1.0 -> lower=-2 upper=+2 effort=30 velocity=1.0

File: src/mobile_manipulator/model/mobile_manipulator.xacro (robot description, xacro)
@@ -292,5 +292,5 @@
   <xacro:Revjoint id="wrist_pitch" trans="0 0 ${length + 0.052 + 0.054}" rpy="0 0 0" parent="wrist_bracket" child="wrist_pitch_motor" axis="1 0 0" l="-2.36344086" u="2.368556533" v="1.0"/>
   <xacro:FxdJoint id="WP_WR" parent="wrist_pitch_motor" child="wrist_roll_motor" />
-  <xacro:Revjoint id="wrist_roll" trans="0 0.02 0.082" rpy="0 0 -1.57" parent="wrist_roll_motor" child="roll_j_plate" axis="1 0 0" l="-3.14" u="+3.14" v="1.0"/>
+  <xacro:Revjoint id="wrist_roll" trans="0 0.02 0.082" rpy="0 0 -1.57" parent="wrist_roll_motor" child="roll_j_plate" axis="1 0 0" l="-2" u="+2" v="1.0"/>
   <xacro:FxdJoint id="roll_plate_gripper" parent="roll_j_plate" child="gripper" />
 </robot>

Commit message: Hurray! Finally IKFast working with URDF for new arm with gripper What made the difference was the axis selection of the gripper link in the URDF ALWAYS REMEMBER TO SOURCE DEVEL AND CATKIN BUILD THRICE ATLEAST!!!!!!!!! some weird shit with catkin
	modified:   .gitignore
	new file:   .vscode/tags
	new file:   src/ikfast_make.sh
	modified:   src/mobile_manipulator/model/mobile_manipulator.dae
	modified:   src/mobile_manipulator/model/mobile_manipulator.urdf
	modified:   src/mobile_manipulator/model/mobile_manipulator.xacro
	modified:   src/mobile_manipulator_moveit_config/config/mobile_manipulator.srdf

File: src/mobile_manipulator/model/mobile_manipulator.urdf (robot description, URDF)
Before this commit: robot mobile_manipulator, 12 links, 11 joints
Joints:
- joint wrist_roll: axis 1 0 0 -> 0 1 0; origin xyz=0 0.02 0.082 rpy=0 0 -1.57 -> xyz=0 0.02 0.082 rpy=0 3.14 0

File: src/mobile_manipulator/model/mobile_manipulator.xacro (robot description, xacro)
@@ -274,11 +274,11 @@
   <link name="roll_j_plate">
     <xacro:roll_j_plate_Inertial trans="0 0 0" rpy="0 0 0"/>
-    <xacro:roll_j_plate_Visual trans="0 0.021 0.048" rpy="0 1.57 3.14"/>
-    <xacro:roll_j_plate_Collision trans="0 0.021 0.048" rpy="0 1.57 3.14"/>
+    <xacro:roll_j_plate_Visual trans="-0.025 0 -0.052" rpy="-1.57 -1.57 0"/>
+    <xacro:roll_j_plate_Collision trans="-0.025 0 -0.052" rpy="-1.57 -1.57 0"/>
   </link>
  <link name="gripper">
     <xacro:gripper_Inertial trans="0 0 0" rpy="0 0 0"/>
-    <xacro:gripper_Visual trans="-0.069 -0.016 0.004" rpy="0 0 1.57"/>
-    <xacro:gripper_Collision trans="-0.069 -0.016 0.004" rpy="0 0 1.57"/>
+    <xacro:gripper_Visual trans="0.008 0.07 -0.009" rpy="0 3.14 0"/>
+    <xacro:gripper_Collision trans="0.008 0.07 -0.009" rpy="0 3.14 0"/>
   </link>
  <!-- JOINTS -->
@@ -292,5 +292,5 @@
   <xacro:Revjoint id="wrist_pitch" trans="0 0 ${length + 0.052 + 0.054}" rpy="0 0 0" parent="wrist_bracket" child="wrist_pitch_motor" axis="1 0 0" l="-2.36344086" u="2.368556533" v="1.0"/>
   <xacro:FxdJoint id="WP_WR" parent="wrist_pitch_motor" child="wrist_roll_motor" />
-  <xacro:Revjoint id="wrist_roll" trans="0 0.02 0.082" rpy="0 0 -1.57" parent="wrist_roll_motor" child="roll_j_plate" axis="1 0 0" l="-2" u="+2" v="1.0"/>
+  <xacro:Revjoint id="wrist_roll" trans="0 0.02 0.082" rpy="0 3.14 0" parent="wrist_roll_motor" child="roll_j_plate" axis="0 1 0" l="-2" u="+2" v="1.0"/>
   <xacro:FxdJoint id="roll_plate_gripper" parent="roll_j_plate" child="gripper" />
 </robot>

Commit message: Added parallel motor setup, yet to test  Author:    Chinmay Khopde <chinmaykhopde@gmail.com> 	modified:   src/mobile_manipulator/model/ikfast61_arm.cpp 	modified:   src/mobile_manipulator/model/mobile_manipulator.urdf 	modified:   src/mobile_manipulator/model/mobile_manipulator.xacro 	modified:   src/mobile_manipulator_ikfast_arm_plugin/src/mobile_manipulator_arm_ikfast_solver.cpp 	modified:   src/mobile_manipulator_moveit_config/.setup_assistant

File: src/mobile_manipulator/model/mobile_manipulator.urdf (robot description, URDF)
Before this commit: robot mobile_manipulator, 12 links, 11 joints
Links:
- link shoulder_pitch_motor: geometry collision box size=0.041 0.0602 0.1480; visual mesh filename=package://mobile_manipulator/meshes/dynamixel_x64series.stl scale=0.001 0.001 0.001

File: src/mobile_manipulator/model/mobile_manipulator.xacro (robot description, xacro)
@@ -36,4 +36,12 @@
     </collision>
 </xacro:macro>
+<xacro:macro name="MXCollision_dual_motor" params="trans rpy">
+    <collision>
+      <origin xyz="${trans}" rpy="${rpy}"/>
+      <geometry>
+        <box size="0.041 0.0602 0.1480"/>
+      </geometry>
+    </collision>
+</xacro:macro>
 <xacro:macro name="AXInertial" params="trans rpy">
   <inertial>
@@ -235,5 +243,5 @@
     <xacro:MXInertial trans="0 0 0" rpy="1.57 -3.14 1.57"/>
     <xacro:MXVisual trans="0 0 0" rpy="1.57 -3.14 1.57"/>
-    <xacro:MXCollision trans="0 0 0" rpy="1.57 -3.14 1.57"/>
+    <xacro:MXCollision_dual_motor trans="0 0 0" rpy="1.57 -3.14 1.57"/>
   </link>
   <link name="biscep">

Commit message: Added whole bot in the urdf, ran moveit setup assistant rebuilt ikFast
---------------------------------------------------------------------------------
TODO :
	* To test on real bot with arm added
---------------------------------------------------------------------------------

Changed and new files -

	new file:   src/mobile_manipulator/meshes/bot.stl
	new file:   src/mobile_manipulator/meshes/mx-64.stl
	modified:   src/mobile_manipulator/model/ikfast61_arm.cpp
	modified:   src/mobile_manipulator/model/mobile_manipulator.xacro
	modified:   src/mobile_manipulator_moveit_config/.setup_assistant
	modified:   src/mobile_manipulator_moveit_config/config/mobile_manipulator.srdf

File: src/mobile_manipulator/model/mobile_manipulator.urdf (robot description, URDF)
Before this commit: robot mobile_manipulator, 12 links, 11 joints
Links:
- added link bot, mass 0.140; collision mesh filename=package://mobile_manipulator/meshes/bot.stl scale=0.001 0.001 0.001; visual mesh filename=package://mobile_manipulator/meshes/bot.stl scale=0.001 0.001 0.001
Joints:
- added joint bot_joint: type fixed, parent bot, child shoulder_yaw_motor
- joint shoulder_yaw: origin xyz=0 0 0.025 rpy=0 0 0 -> xyz=0 0.188 0.2577 rpy=0 0 0

File: src/mobile_manipulator/model/mobile_manipulator.xacro (robot description, xacro)
@@ -36,4 +36,28 @@
     </collision>
 </xacro:macro>
+<xacro:macro name="BotInertial" params="trans rpy">
+  <inertial>
+    <origin xyz="${trans}" rpy="${rpy}" />
+    <mass value="0.140" />
+    <inertia ixx="0.000050799110" ixy="0.0" ixz="0.0" iyy="0.00002857215" iyz="0.00000051457" izz="0.000043394" />
+  </inertial>
+</xacro:macro>
+<xacro:macro name="BotVisual" params="trans rpy">
+  <visual>
+    <origin xyz="${trans}" rpy="${rpy}"/>
+    <geometry>
+      <mesh filename="package://mobile_manipulator/meshes/bot.stl" scale="0.001 0.001 0.001"/>
+    </geometry>
+    <material name="white"/>
+  </visual>
+</xacro:macro>
+<xacro:macro name="BotCollision" params="trans rpy">
+    <collision>
+      <origin xyz="${trans}" rpy="${rpy}"/>
+      <geometry>
+        <mesh filename="package://mobile_manipulator/meshes/bot.stl" scale="0.001 0.001 0.001"/>
+      </geometry>
+    </collision>
+</xacro:macro>
 <xacro:macro name="MXCollision_dual_motor" params="trans rpy">
     <collision>
@@ -230,8 +254,13 @@
 </xacro:macro>
 <!-- LINKS -->
+  <link name="bot">
+    <xacro:BotInertial trans="0 0 0" rpy="0 0 0 "/>
+    <xacro:BotVisual trans="0 0 0" rpy="0 0 0 "/>
+    <xacro:BotCollision trans="0 0 0" rpy="0 0 0"/>
+  </link>
   <link name="shoulder_yaw_motor">
     <xacro:MXInertial trans="0 0 0" rpy="0 0 0 "/>
-    <xacro:MXVisual trans="0 0 0" rpy="0 0 0 "/>
-    <xacro:MXCollision trans="0 0 0" rpy="0 0 0"/>
+    <xacro:MXVisual trans="0 0.188 0.2349" rpy="0 0 0 "/>
+    <xacro:MXCollision trans="0 0.188 0.2349" rpy="0 0 0"/>
   </link>
   <link name="shoulder_bracket">
@@ -290,6 +319,8 @@
     <xacro:gripper_Collision trans="0.008 0.07 -0.009" rpy="0 3.14 0"/>
   </link>
- <!-- JOINTS -->
-  <xacro:Revjoint id="shoulder_yaw" trans="0 0 0.025" rpy="0 0 0" parent="shoulder_yaw_motor" child="shoulder_bracket" axis="0 0 1" l="-3.0357" u="3.24426" v="1.0"/>
+ <!-- JOINTS -->3
+  <xacro:FxdJoint id="bot_joint" parent="bot" child="shoulder_yaw_motor"/>
+  <xacro:Revjoint id="shoulder_yaw" trans="0 0.188 0.2577" rpy="0 0 0" parent="shoulder_yaw_motor" child="shoulder_bracket" axis="0 0 1" l="-3.0357" u="3.24426" v="1.0"/>
+  <!-- 0 0 0.025 -->
   <xacro:Revjoint id="shoulder_pitch" trans="0 0 0.035" rpy="0 0 0" parent="shoulder_bracket" child="shoulder_pitch_motor" axis="1 0 0" l="-1.973232422" u="1.916503906" v="1.0"/>
   <xacro:FxdJoint id="s1_l2" parent="shoulder_pitch_motor" child="biscep"/>

Commit message: Intermediate commit for 6DOF arm *Added new wrist yaw motor and generated the ikfast solution *Made changes to the dynamixel controllers and state_publishers *Dynamixels and state_publishers work, interactive marker in Rviz and fk, ik do not *Will try ikfast again by making axis changes of tool in URDF

File: src/mobile_manipulator/model/mobile_manipulator.urdf (robot description, URDF)
Before this commit: robot mobile_manipulator, 13 links, 12 joints
Links:
- added link wrist_yaw_motor, mass 0.05573; collision box size=0.032 0.04 0.05; visual mesh filename=package://mobile_manipulator/meshes/AX-12_18A - dynamixel_A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 scale=0.001 0.001 0.001
Joints:
- removed joint WP_WR
- added joint WP_WY: type fixed, parent wrist_pitch_motor, child wrist_yaw_motor
- added joint wrist_yaw: type revolute, parent wrist_yaw_motor, child wrist_roll_motor, origin xyz=0 0.02 0.058 rpy=0 0 0, axis 0 0 1, limit lower=-2.36344086 upper=2.368556533 effort=30 velocity=1.0
- joint wrist_roll: origin xyz=0 0.02 0.082 rpy=0 3.14 0 -> xyz=0 0 0.058 rpy=0 0 0

File: src/mobile_manipulator/model/mobile_manipulator.xacro (robot description, xacro)
@@ -304,17 +304,29 @@
     <xacro:AXCollision trans="0 0 0" rpy="-1.57 0 -1.57"/>
   </link>
+  <!-- ADD FLAT TINY BOX HERE -->
+  <!-- <link name="new_bracket">
+    <xacro:AxBracketInertial trans="0 0 ${0.052+length+0.054}" rpy="1.57 0 1.57"/>
+    <xacro:AxBracketVisual trans="0 0 ${0.052+length+0.054}" rpy="1.57 0 1.57"/>
+    <xacro:AxBracketCollision trans="0 0 ${0.052+length+0.054}" rpy="1.57 0 1.57"/>
+  </link>
+   -->
+  <link name="wrist_yaw_motor">
+    <xacro:AXInertial trans="0 0 0.058" rpy="0 3.14 0"/>
+    <xacro:AXVisual trans="0 0.018 0.058" rpy="0 3.14 0"/>
+    <xacro:AXCollision trans="0 0 0.058" rpy="-1.57 3.14 0"/>
+  </link>
   <link name="wrist_roll_motor">
-    <xacro:AXInertial trans="0 0 0.078" rpy="-1.57 3.14 0"/>
-    <xacro:AXVisual trans="0 0 0.078" rpy="-1.57 3.14 0"/>
-    <xacro:AXCollision trans="0 0 0.078" rpy="-1.57 3.14 0"/>
+    <xacro:AXInertial trans="0 0 0.058" rpy="-1.57 3.14 0"/>
+    <xacro:AXVisual trans="0 0 0.058" rpy="-1.57 3.14 0"/>
+    <xacro:AXCollision trans="0 0 0.058" rpy="-1.57 3.14 0"/>
   </link>
   <link name="roll_j_plate">
     <xacro:roll_j_plate_Inertial trans="0 0 0" rpy="0 0 0"/>
-    <xacro:roll_j_plate_Visual trans="-0.025 0 -0.052" rpy="-1.57 -1.57 0"/>
+    <xacro:roll_j_plate_Visual trans="0.02 0.023 0.053" rpy="-1.57 1.57 0"/>
     <xacro:roll_j_plate_Collision trans="-0.025 0 -0.052" rpy="-1.57 -1.57 0"/>
   </link>
  <link name="gripper">
     <xacro:gripper_Inertial trans="0 0 0" rpy="0 0 0"/>
-    <xacro:gripper_Visual trans="0.008 0.07 -0.009" rpy="0 3.14 0"/>
+    <xacro:gripper_Visual trans="-0.019 0.092 0.002" rpy="0 0 0"/>
     <xacro:gripper_Collision trans="0.008 0.07 -0.009" rpy="0 3.14 0"/>
   </link>
@@ -330,6 +342,9 @@
   <xacro:FxdJoint id="l3_l3B" parent="forearm" child="wrist_bracket"/>
   <xacro:Revjoint id="wrist_pitch" trans="0 0 ${length + 0.052 + 0.054}" rpy="0 0 0" parent="wrist_bracket" child="wrist_pitch_motor" axis="1 0 0" l="-2.36344086" u="2.368556533" v="1.0"/>
-  <xacro:FxdJoint id="WP_WR" parent="wrist_pitch_motor" child="wrist_roll_motor" />
-  <xacro:Revjoint id="wrist_roll" trans="0 0.02 0.082" rpy="0 3.14 0" parent="wrist_roll_motor" child="roll_j_plate" axis="0 1 0" l="-2" u="+2" v="1.0"/>
+  <xacro:FxdJoint id="WP_WY" parent="wrist_pitch_motor" child="wrist_yaw_motor" />
+  <xacro:Revjoint id="wrist_yaw" trans="0 0.02 0.058" rpy="0 0 0" parent="wrist_yaw_motor" child="wrist_roll_motor" axis="0 0 1" l="-2.36344086" u="2.368556533" v="1.0"/>
+  <xacro:Revjoint id="wrist_roll" trans="0 0 0.058" rpy="0 0 0" parent="wrist_roll_motor" child="roll_j_plate" axis="0 1 0" l="-2" u="+2" v="1.0"/>
   <xacro:FxdJoint id="roll_plate_gripper" parent="roll_j_plate" child="gripper" />
 </robot>
+<!-- 0 0.018 0.06 -->
+<!-- 0 0.02 0.082 -->

Commit message: *IKFast succesfull for 6DOF arm. The interactive marker is now moving in RViz *Some new issue with "invalid initial state on planning"

File: src/mobile_manipulator/model/mobile_manipulator.urdf (robot description, URDF)
Before this commit: robot mobile_manipulator, 14 links, 13 joints
Links:
- removed link bot
Joints:
- removed joint bot_joint
- joint shoulder_yaw: origin xyz=0 0.188 0.2577 rpy=0 0 0 -> xyz=0 0 0 rpy=0 0 0

File: src/mobile_manipulator/model/mobile_manipulator.xacro (robot description, xacro)
@@ -254,9 +254,9 @@
 </xacro:macro>
 <!-- LINKS -->
-  <link name="bot">
+  <!-- <link name="bot">
     <xacro:BotInertial trans="0 0 0" rpy="0 0 0 "/>
     <xacro:BotVisual trans="0 0 0" rpy="0 0 0 "/>
     <xacro:BotCollision trans="0 0 0" rpy="0 0 0"/>
-  </link>
+  </link> -->
   <link name="shoulder_yaw_motor">
     <xacro:MXInertial trans="0 0 0" rpy="0 0 0 "/>
@@ -332,6 +332,6 @@
   </link>
  <!-- JOINTS -->
-  <xacro:FxdJoint id="bot_joint" parent="bot" child="shoulder_yaw_motor"/>
-  <xacro:Revjoint id="shoulder_yaw" trans="0 0.188 0.2577" rpy="0 0 0" parent="shoulder_yaw_motor" child="shoulder_bracket" axis="0 0 1" l="-3.0357" u="3.24426" v="1.0"/>
+  <!-- <xacro:FxdJoint id="bot_joint" parent="bot" child="shoulder_yaw_motor"/> -->
+  <xacro:Revjoint id="shoulder_yaw" trans="0 0 0" rpy="0 0 0" parent="shoulder_yaw_motor" child="shoulder_bracket" axis="0 0 1" l="-3.0357" u="3.24426" v="1.0"/>
   <!-- 0 0 0.025 -->
   <xacro:Revjoint id="shoulder_pitch" trans="0 0 0.035" rpy="0 0 0" parent="shoulder_bracket" child="shoulder_pitch_motor" axis="1 0 0" l="-1.973232422" u="1.916503906" v="1.0"/>
@@ -349,2 +349,3 @@
 <!-- 0 0.018 0.06 -->
 <!-- 0 0.02 0.082 -->
+<!--0vghvg  0.188 0.2577 -->

Commit message: 6dof working. Made changes to collision parameters

File: src/mobile_manipulator/model/mobile_manipulator.urdf (robot description, URDF)
Before this commit: robot mobile_manipulator, 13 links, 12 joints
Links:
- link shoulder_pitch_motor: geometry collision box size=0.041 0.0402 0.0611; visual mesh filename=package://mobile_manipulator/meshes/dynamixel_x64series.stl scale=0.001 0.001 0.001

File: src/mobile_manipulator/model/mobile_manipulator.xacro (robot description, xacro)
@@ -261,6 +261,6 @@
   <link name="shoulder_yaw_motor">
     <xacro:MXInertial trans="0 0 0" rpy="0 0 0 "/>
-    <xacro:MXVisual trans="0 0.188 0.2349" rpy="0 0 0 "/>
-    <xacro:MXCollision trans="0 0.188 0.2349" rpy="0 0 0"/>
+    <xacro:MXVisual trans="0 0 -0.027" rpy="0 0 0 "/>
+    <xacro:MXCollision trans="0 0 -0.027" rpy="0 0 0"/>
   </link>
   <link name="shoulder_bracket">
@@ -272,5 +272,5 @@
     <xacro:MXInertial trans="0 0 0" rpy="1.57 -3.14 1.57"/>
     <xacro:MXVisual trans="0 0 0" rpy="1.57 -3.14 1.57"/>
-    <xacro:MXCollision_dual_motor trans="0 0 0" rpy="1.57 -3.14 1.57"/>
+    <xacro:MXCollision trans="0 0 0" rpy="1.57 -3.14 1.57"/>
   </link>
   <link name="biscep">
@@ -312,7 +312,7 @@
    -->
   <link name="wrist_yaw_motor">
-    <xacro:AXInertial trans="0 0 0.058" rpy="0 3.14 0"/>
+    <xacro:AXInertial trans="0 0.018 0.058" rpy="0 3.14 0"/>
     <xacro:AXVisual trans="0 0.018 0.058" rpy="0 3.14 0"/>
-    <xacro:AXCollision trans="0 0 0.058" rpy="-1.57 3.14 0"/>
+    <xacro:AXCollision trans="0 0.018 0.058" rpy="0 3.14 0"/>
   </link>
   <link name="wrist_roll_motor">
@@ -329,5 +329,5 @@
     <xacro:gripper_Inertial trans="0 0 0" rpy="0 0 0"/>
     <xacro:gripper_Visual trans="-0.019 0.092 0.002" rpy="0 0 0"/>
-    <xacro:gripper_Collision trans="0.008 0.07 -0.009" rpy="0 3.14 0"/>
+    <xacro:gripper_Collision trans="-0.019 0.092 0.002" rpy="0 0 0"/>
   </link>
  <!-- JOINTS -->
