Commit message: -Some progress with the 6dof manipulator -Completely redesigned the xacro file and also added the dual motor assembly -The interactive marker moves smoothly, but the wrist yaw ring does not. -Although move it does move the yaw motor for certain goals

File: src/mobile_manipulator/model/mobile_manipulator.urdf (robot description, URDF)
Before this commit: robot mobile_manipulator, 13 links, 12 joints
Links:
- added link bot, mass 0.140; collision mesh filename=package://mobile_manipulator/meshes/bot.stl scale=0.001 0.001 0.001; visual mesh filename=package://mobile_manipulator/meshes/bot.stl scale=0.001 0.001 0.001
- link shoulder_bracket: geometry collision mesh filename=package://mobile_manipulator/meshes/Dual_bracket.stl scale=0.0001 0.0001 0.0001; visual mesh filename=package://mobile_manipulator/meshes/Dual_bracket.stl scale=0.0001 0.0001 0.0001
- link shoulder_pitch_motor: mass 0.140 -> 0.00712; geometry collision mesh filename=package://mobile_manipulator/meshes/ParallelMotors.stl scale=0.001 0.001 0.001; visual mesh filename=package://mobile_manipulator/meshes/ParallelMotors.stl scale=0.001 0.001 0.001
Joints:
- removed joint shoulder_pitch
- removed joint shoulder_yaw
- added joint bot_to_shoulder_yaw_motor_fxd: type fixed, parent bot, child shoulder_yaw_motor, origin xyz=0 0.1722 0.256 rpy=0 0 0
- added joint shoulder_pitch_joint_rev: type revolute, parent shoulder_bracket, child shoulder_pitch_motor, origin xyz=0 0 0.04 rpy=0 1.57 0, axis 0 0 1, limit lower=-1.973232422 upper=1.916503906 effort=30 velocity=1.0
- added joint shoulder_yaw_joint_rev: type revolute, parent shoulder_yaw_motor, child shoulder_bracket, origin xyz=0 0 0 rpy=0 0 0, axis 0 0 1, limit lower=-3.0357 upper=3.24426 effort=30 velocity=1.0
- joint WP_WY: origin (none) -> xyz=-0.061 0.02 0 rpy=0 -1.57 0
- joint e_l3: origin (none) -> xyz=0 0 0 rpy=0 0 0
- joint elbow: axis 1 0 0 -> 0 0 1; origin xyz=0 0 0.186 rpy=0 0 0 -> xyz=-0.186 0 0 rpy=0 0 0
- joint l2_l2B: origin (none) -> xyz=0 0 0 rpy=0 0 0
- joint l3_l3B: origin (none) -> xyz=0 0 0 rpy=0 0 0
- joint roll_plate_gripper: origin (none) -> xyz=0 0 0 rpy=0 0 0
- joint s1_l2: origin (none) -> xyz=0 0 0 rpy=0 0 0
- joint wrist_pitch: axis 1 0 0 -> 0 0 1; origin xyz=0 0 0.202 rpy=0 0 0 -> xyz=-0.202 0 0 rpy=0 0 0
- joint wrist_roll: axis 0 1 0 -> 0 0 1; origin xyz=0 0 0.058 rpy=0 0 0 -> xyz=0 0 0 rpy=0 0 0
- joint wrist_yaw: axis 0 0 1 -> 0 1 0; origin xyz=0 0.02 0.058 rpy=0 0 0 -> xyz=0 0 0.065 rpy=-1.57 0 0

File: src/mobile_manipulator/model/mobile_manipulator.xacro (robot description, xacro)
@@ -116,4 +116,52 @@
     </collision>
 </xacro:macro>
+<xacro:macro name="Dual_Bracket_Inertial" params="trans rpy">
+  <inertial>
+    <origin xyz="${trans}" rpy="${rpy}"/>
+    <mass value="0.00712" />
+    <inertia ixx="0.00000174511" iyy="0.00000379922" ixz="0.0" ixy="0.0" iyz="0.0" izz="0.00000357521" />
+  </inertial>
+</xacro:macro>
+<xacro:macro name="Dual_Bracket_Visual" params="trans rpy">
+  <visual>
+    <origin xyz="${trans}" rpy="${rpy}"/>
+    <geometry>
+      <mesh filename="package://mobile_manipulator/meshes/Dual_bracket.stl" scale="0.0001 0.0001 0.0001" />
+    </geometry>
+    <material name="white"/>
+  </visual>
+</xacro:macro>
+<xacro:macro name="Dual_Bracket_Collision" params="trans rpy">
+    <collision>
+      <origin xyz="${trans}" rpy="${rpy}"/>
+      <geometry>
+        <mesh filename="package://mobile_manipulator/meshes/Dual_bracket.stl" scale="0.0001 0.0001 0.0001"/>
+      </geometry>
+    </collision>
+</xacro:macro>
+<xacro:macro name="Parallel_Motor_Inertial" params="trans rpy">
+  <inertial>
+    <origin xyz="${trans}" rpy="${rpy}"/>
+    <mass value="0.00712" />
+    <inertia ixx="0.00000174511" iyy="0.00000379922" ixz="0.0" ixy="0.0" iyz="0.0" izz="0.00000357521" />
+  </inertial>
+</xacro:macro>
+<xacro:macro name="Parallel_Motor_Visual" params="trans rpy">
+  <visual>
+    <origin xyz="${trans}" rpy="${rpy}"/>
+    <geometry>
+      <mesh filename="package://mobile_manipulator/meshes/ParallelMotors.stl" scale="0.001 0.001 0.001" />
+    </geometry>
+    <material name="white"/>
+  </visual>
+</xacro:macro>
+<xacro:macro name="Parallel_Motor_Collision" params="trans rpy">
+    <collision>
+      <origin xyz="${trans}" rpy="${rpy}"/>
+      <geometry>
+        <mesh filename="package://mobile_manipulator/meshes/ParallelMotors.stl" scale="0.001 0.001 0.001"/>
+      </geometry>
+    </collision>
+</xacro:macro>
 <xacro:macro name="AxBracketInertial" params="trans rpy">
   <inertial>
@@ -223,8 +271,9 @@
     </joint>
 </xacro:macro>
-<xacro:macro name="FxdJoint" params="id parent child">
+<xacro:macro name="FxdJoint" params="id trans rpy parent child ">
     <joint name="${id}" type="fixed">
       <parent link="${parent}"/>
       <child link="${child}"/>
+       <origin xyz="${trans}" rpy="${rpy}"/>
     </joint>
 </xacro:macro>
@@ -254,96 +303,90 @@
 </xacro:macro>
 <!-- LINKS -->
-  <!-- <link name="bot">
+  <link name="bot">
     <xacro:BotInertial trans="0 0 0" rpy="0 0 0 "/>
     <xacro:BotVisual trans="0 0 0" rpy="0 0 0 "/>
     <xacro:BotCollision trans="0 0 0" rpy="0 0 0"/>
-  </link> -->
+  </link>
   <link name="shoulder_yaw_motor">
-    <xacro:MXInertial trans="0 0 0" rpy="0 0 0 "/>
-    <xacro:MXVisual trans="0 0 -0.027" rpy="0 0 0 "/>
+    <xacro:MXInertial trans="0 0 -0.027" rpy="0 0 0"/>
+    <xacro:MXVisual trans="0 0 -0.027" rpy="0 0 0"/>
     <xacro:MXCollision trans="0 0 -0.027" rpy="0 0 0"/>
   </link>
   <link name="shoulder_bracket">
-    <xacro:BracketInertial trans="0 0 0.025" rpy="0 3.14 0 "/>
-    <xacro:BracketVisual trans="0 0 0" rpy="0 3.14 0 "/>
-    <xacro:BracketCollision trans="0 0 0" rpy="0 3.14 0 "/>
+    <xacro:Dual_Bracket_Inertial trans="0 0 -0.005" rpy="0 0 1.57"/>
+    <xacro:Dual_Bracket_Visual trans="0 0 -0.005" rpy="0 0 1.57"/>
+    <xacro:Dual_Bracket_Collision trans="0 0 -0.005" rpy="0 0 1.57"/>
   </link>
   <link name="shoulder_pitch_motor">
-    <xacro:MXInertial trans="0 0 0" rpy="1.57 -3.14 1.57"/>
-    <xacro:MXVisual trans="0 0 0" rpy="1.57 -3.14 1.57"/>
-    <xacro:MXCollision trans="0 0 0" rpy="1.57 -3.14 1.57"/>
+    <xacro:Parallel_Motor_Inertial trans="0 0 0" rpy="0 0 -1.57"/>
+    <xacro:Parallel_Motor_Visual trans="0 0 0" rpy="0 0 -1.57"/>
+    <xacro:Parallel_Motor_Collision trans="0 0 0" rpy="0 0 -1.57"/>
   </link>
   <link name="biscep">
-    <xacro:LinkInertial trans="0 0 ${0.051+(length/2)}" rpy="0 0 0" />
-    <xacro:LinkVisual trans="0 0 ${0.051+(length/2)}" rpy="0 0 0" />
-    <xacro:LinkCollision trans="0 0 ${0.051+(length/2)}" rpy="0 0 0" />
-  </link>
-  <link name="elbow_bracket">
-    <xacro:BracketInertial trans="0 0 ${0.052+length}" rpy="0 3.14 0"/>
-    <xacro:BracketVisual trans="0 0 ${0.052+length}" rpy="0 3.14 0"/>
-    <xacro:BracketCollision trans="0 0 ${0.052+length}" rpy="0 3.14 0"/>
-  </link>
-  <link name="elbow_motor">
-    <xacro:MXInertial trans="0 0 0" rpy="1.57 0 0"/>
-    <xacro:MXVisual trans="0 0 0" rpy="1.57 3.14 -1.57"/>
-    <xacro:MXCollision trans="0 0 0" rpy="1.57 3.14 -1.57"/>
+    <xacro:LinkInertial trans="-${0.0575+(length/2)} 0 0" rpy="0 -1.57 0" />
+    <xacro:LinkVisual trans="-${0.0575+(length/2)} 0 0" rpy="0 -1.57 0" />
+    <xacro:LinkCollision trans="-${0.0575+(length/2)} 0 0" rpy="0 -1.57 0" />
+  </link>
+   <link name="elbow_bracket">
+    <xacro:BracketInertial trans="-${0.062+length} 0 0" rpy="0 1.57 0"/>
+    <xacro:BracketVisual trans="-${0.062+length} 0 0" rpy="0 1.57 0"/>
+    <xacro:BracketCollision trans="-${0.062+length} 0 0" rpy="0 1.57 0"/>
+  </link>
+    <link name="elbow_motor">
+    <xacro:MXInertial trans="0 0 0" rpy="0 0 -1.57"/>
+    <xacro:MXVisual trans="0 0 0" rpy="0 0 -1.57"/>
+    <xacro:MXCollision trans="0 0 0" rpy="0 0 -1.57"/>
   </link>
   <link name="forearm">
-    <xacro:LinkInertial trans="0 0 ${0.052+(length/2)}" rpy="0 0 0" />
-    <xacro:LinkVisual trans="0 0 ${0.052+(length/2)}" rpy="0 0 0" />
-    <xacro:LinkCollision trans="0 0 ${0.052+(length/2)}" rpy="0 0 0" />
+    <xacro:LinkInertial trans="-${0.047+(length/2)} 0 0" rpy="0 -1.57 0" />
+    <xacro:LinkVisual trans="-${0.047+(length/2)} 0 0" rpy="0 -1.57 0" />
+    <xacro:LinkCollision trans="-${0.047+(length/2)} 0 0" rpy="0 -1.57 0" />
   </link>
   <link name="wrist_bracket">
-    <xacro:AxBracketInertial trans="0 0 ${0.052+length+0.054}" rpy="1.57 0 1.57"/>
-    <xacro:AxBracketVisual trans="0 0 ${0.052+length+0.054}" rpy="1.57 0 1.57"/>
-    <xacro:AxBracketCollision trans="0 0 ${0.052+length+0.054}" rpy="1.57 0 1.57"/>
+    <xacro:AxBracketInertial trans="-${0.047+length+0.054} 0 0" rpy="0 0 1.57"/>
+    <xacro:AxBracketVisual trans="-${0.047+length+0.054} 0 0" rpy="0 0 1.57"/>
+    <xacro:AxBracketCollision trans="-${0.047+length+0.054} 0 0" rpy="0 0 1.57"/>
   </link>
   <link name="wrist_pitch_motor">
-    <xacro:AXInertial trans="0 0 0" rpy="-1.57 0 -1.57"/>
-    <xacro:AXVisual trans="0 0 0" rpy="-1.57 0 -1.57"/>
-    <xacro:AXCollision trans="0 0 0" rpy="-1.57 0 -1.57"/>
-  </link>
-  <!-- ADD FLAT TINY BOX HERE -->
-  <!-- <link name="new_bracket">
-    <xacro:AxBracketInertial trans="0 0 ${0.052+length+0.054}" rpy="1.57 0 1.57"/>
-    <xacro:AxBracketVisual trans="0 0 ${0.052+length+0.054}" rpy="1.57 0 1.57"/>
-    <xacro:AxBracketCollision trans="0 0 ${0.052+length+0.054}" rpy="1.57 0 1.57"/>
-  </link>
-   -->
+    <xacro:AXInertial trans="0.005 0 0" rpy="0 0 -1.57"/>
+    <xacro:AXVisual trans="0.005 0 0" rpy="0 0 -1.57"/>
+    <xacro:AXCollision trans="0.005 0 0" rpy="0 0 -1.57"/>
+  </link>
   <link name="wrist_yaw_motor">
-    <xacro:AXInertial trans="0 0.018 0.058" rpy="0 3.14 0"/>
-    <xacro:AXVisual trans="0 0.018 0.058" rpy="0 3.14 0"/>
-    <xacro:AXCollision trans="0 0.018 0.058" rpy="0 3.14 0"/>
+    <xacro:AXInertial trans="0 0 0" rpy="0 0 0"/>
+    <xacro:AXVisual trans="0 0 0" rpy="0 0 0"/>
+    <xacro:AXCollision trans="0 0 0" rpy="0 0 0"/>
   </link>
   <link name="wrist_roll_motor">
-    <xacro:AXInertial trans="0 0 0.058" rpy="-1.57 3.14 0"/>
-    <xacro:AXVisual trans="0 0 0.058" rpy="-1.57 3.14 0"/>
-    <xacro:AXCollision trans="0 0 0.058" rpy="-1.57 3.14 0"/>
+    <xacro:AXInertial trans="0 0 0" rpy="0 0 3.14"/>
+    <xacro:AXVisual trans="0 0 0" rpy="0 0 3.14"/>
+    <xacro:AXCollision trans="0 0 0" rpy="0 0 3.14"/>
   </link>
   <link name="roll_j_plate">
-    <xacro:roll_j_plate_Inertial trans="0 0 0" rpy="0 0 0"/>
-    <xacro:roll_j_plate_Visual trans="0.02 0.023 0.053" rpy="-1.57 1.57 0"/>
-    <xacro:roll_j_plate_Collision trans="-0.025 0 -0.052" rpy="-1.57 -1.57 0"/>
+    <xacro:roll_j_plate_Inertial trans="0.02 -0.053 0.023" rpy="0 0 1.57"/>
+    <xacro:roll_j_plate_Visual trans="0.02 -0.053 0.023" rpy="0 0 1.57"/>
+    <xacro:roll_j_plate_Collision trans="0.02 -0.053 0.023" rpy="0 0 1.57"/>
   </link>
  <link name="gripper">
-    <xacro:gripper_Inertial trans="0 0 0" rpy="0 0 0"/>
-    <xacro:gripper_Visual trans="-0.019 0.092 0.002" rpy="0 0 0"/>
-    <xacro:gripper_Collision trans="-0.019 0.092 0.002" rpy="0 0 0"/>
-  </link>
+    <xacro:gripper_Inertial trans="-0.01 -0.011 0.092" rpy="1.57 0 0"/>
+    <xacro:gripper_Visual trans="-0.01 -0.011 0.092" rpy="1.57 0 0"/>
+    <xacro:gripper_Collision trans="-0.01 -0.011 0.092" rpy="1.57 0 0"/>
+  </link>
+  <!-- -0.019 0.092 0.002 -->
  <!-- JOINTS -->
-  <!-- <xacro:FxdJoint id="bot_joint" parent="bot" child="shoulder_yaw_motor"/> -->
-  <xacro:Revjoint id="shoulder_yaw" trans="0 0 0" rpy="0 0 0" parent="shoulder_yaw_motor" child="shoulder_bracket" axis="0 0 1" l="-3.0357" u="3.24426" v="1.0"/>
+  <xacro:FxdJoint id="bot_to_shoulder_yaw_motor_fxd" trans="0 0.1722 0.256" rpy="0 0 0" parent="bot" child="shoulder_yaw_motor"/>
+  <xacro:Revjoint id="shoulder_yaw_joint_rev" trans="0 0 0" rpy="0 0 0" parent="shoulder_yaw_motor" child="shoulder_bracket" axis="0 0 1" l="-3.0357" u="3.24426" v="1.0"/>
   <!-- 0 0 0.025 -->
-  <xacro:Revjoint id="shoulder_pitch" trans="0 0 0.035" rpy="0 0 0" parent="shoulder_bracket" child="shoulder_pitch_motor" axis="1 0 0" l="-1.973232422" u="1.916503906" v="1.0"/>
-  <xacro:FxdJoint id="s1_l2" parent="shoulder_pitch_motor" child="biscep"/>
-  <xacro:FxdJoint id="l2_l2B" parent="biscep" child="elbow_bracket"/>
-  <xacro:Revjoint id="elbow" trans="0 0 ${0.052 + (length) + 0.038}" rpy="0 0 0" parent="elbow_bracket" child="elbow_motor" axis="1 0 0" l="-1.99" u="1.971699219" v="1.0"/>
-  <xacro:FxdJoint id="e_l3" parent="elbow_motor" child="forearm"/>
-  <xacro:FxdJoint id="l3_l3B" parent="forearm" child="wrist_bracket"/>
-  <xacro:Revjoint id="wrist_pitch" trans="0 0 ${length + 0.052 + 0.054}" rpy="0 0 0" parent="wrist_bracket" child="wrist_pitch_motor" axis="1 0 0" l="-2.36344086" u="2.368556533" v="1.0"/>
-  <xacro:FxdJoint id="WP_WY" parent="wrist_pitch_motor" child="wrist_yaw_motor" />
-  <xacro:Revjoint id="wrist_yaw" trans="0 0.02 0.058" rpy="0 0 0" parent="wrist_yaw_motor" child="wrist_roll_motor" axis="0 0 1" l="-2.36344086" u="2.368556533" v="1.0"/>
-  <xacro:Revjoint id="wrist_roll" trans="0 0 0.058" rpy="0 0 0" parent="wrist_roll_motor" child="roll_j_plate" axis="0 1 0" l="-2" u="+2" v="1.0"/>
-  <xacro:FxdJoint id="roll_plate_gripper" parent="roll_j_plate" child="gripper" />
+  <xacro:Revjoint id="shoulder_pitch_joint_rev" trans="0 0 0.04" rpy="0 1.57 0" parent="shoulder_bracket" child="shoulder_pitch_motor" axis="0 0 1" l="-1.973232422" u="1.916503906" v="1.0"/>
+  <xacro:FxdJoint id="s1_l2" parent="shoulder_pitch_motor" child="biscep" trans="0 0 0" rpy="0 0 0" />
+  <xacro:FxdJoint id="l2_l2B" parent="biscep" child="elbow_bracket" trans="0 0 0" rpy="0 0 0" />
+  <xacro:Revjoint id="elbow" trans="-${0.052 + (length) + 0.038} 0 0" rpy="0 0 0" parent="elbow_bracket" child="elbow_motor" axis="0 0 1" l="-1.99" u="1.971699219" v="1.0"/>
+  <xacro:FxdJoint id="e_l3" parent="elbow_motor" child="forearm" trans="0 0 0" rpy="0 0 0"/>
+  <xacro:FxdJoint id="l3_l3B" parent="forearm" child="wrist_bracket" trans="0 0 0" rpy="0 0 0"/>
+  <xacro:Revjoint id="wrist_pitch" trans="-${length + 0.052 + 0.054} 0 0" rpy="0 0 0" parent="wrist_bracket" child="wrist_pitch_motor" axis="0 0 1" l="-2.36344086" u="2.368556533" v="1.0"/>
+  <xacro:FxdJoint id="WP_WY" parent="wrist_pitch_motor" child="wrist_yaw_motor" trans="-0.061 0.02 0" rpy="0 -1.57 0"/>
+  <xacro:Revjoint id="wrist_yaw" trans="0 0 0.065" rpy="-1.57 0 0" parent="wrist_yaw_motor" child="wrist_roll_motor" axis="0 1 0" l="-2.36344086" u="2.368556533" v="1.0"/>
+  <xacro:Revjoint id="wrist_roll" trans="0 0 0" rpy="0 0 0" parent="wrist_roll_motor" child="roll_j_plate" axis="0 0 1" l="-2" u="+2" v="1.0"/>
+  <xacro:FxdJoint id="roll_plate_gripper" parent="roll_j_plate" child="gripper" trans="0 0 0" rpy="0 0 0"/>
 </robot>
 <!-- 0 0.018 0.06 -->

Commit message: Pausing 6DOF arm, returning to 5DOF

File: src/mobile_manipulator/model/mobile_manipulator.urdf (robot description, URDF)
Before this commit: robot mobile_manipulator, 14 links, 13 joints
Joints:
- joint wrist_roll: axis 0 0 1 -> 1 0 0; origin xyz=0 0 0 rpy=0 0 0 -> xyz=0 0 0 rpy=0 0 1.57
- joint wrist_yaw: axis 0 1 0 -> 0 0 1; origin xyz=0 0 0.065 rpy=-1.57 0 0 -> xyz=0 0 0.065 rpy=0 0 0

File: src/mobile_manipulator/model/mobile_manipulator.xacro (robot description, xacro)
@@ -359,20 +359,21 @@
   </link>
   <link name="wrist_roll_motor">
-    <xacro:AXInertial trans="0 0 0" rpy="0 0 3.14"/>
-    <xacro:AXVisual trans="0 0 0" rpy="0 0 3.14"/>
-    <xacro:AXCollision trans="0 0 0" rpy="0 0 3.14"/>
+    <xacro:AXInertial trans="0 0 0" rpy="1.57 0 0"/>
+    <xacro:AXVisual trans="0 0 0" rpy="1.57 0 0"/>
+    <xacro:AXCollision trans="0 0 0" rpy="1.57 0 0"/>
   </link>
   <link name="roll_j_plate">
-    <xacro:roll_j_plate_Inertial trans="0.02 -0.053 0.023" rpy="0 0 1.57"/>
-    <xacro:roll_j_plate_Visual trans="0.02 -0.053 0.023" rpy="0 0 1.57"/>
-    <xacro:roll_j_plate_Collision trans="0.02 -0.053 0.023" rpy="0 0 1.57"/>
+    <xacro:roll_j_plate_Inertial trans="0.02 0.023 0.053" rpy="0 1.57 1.57"/>
+    <xacro:roll_j_plate_Visual trans="0.02 -0.023 0.053" rpy="0 1.57 0"/>
+    <xacro:roll_j_plate_Collision trans="0.02 0.023 0.053" rpy="0 1.57 1.57"/>
   </link>
  <link name="gripper">
-    <xacro:gripper_Inertial trans="-0.01 -0.011 0.092" rpy="1.57 0 0"/>
-    <xacro:gripper_Visual trans="-0.01 -0.011 0.092" rpy="1.57 0 0"/>
-    <xacro:gripper_Collision trans="-0.01 -0.011 0.092" rpy="1.57 0 0"/>
+    <xacro:gripper_Inertial trans="-0.011 0.092 0.01" rpy="0 0 0"/>
+    <xacro:gripper_Visual trans="0.092 0.01 0.011" rpy="0 0 -1.57"/>
+    <xacro:gripper_Collision trans="-0.011 0.092 0.01" rpy="0 0 0"/>
   </link>
   <!-- -0.019 0.092 0.002 -->
  <!-- JOINTS -->
+  <!-- <xacro:FxdJoint id="bot_to_map" trans="0 0 0" rpy="0 0 0" parent="map" child="bot"/>  -->
   <xacro:FxdJoint id="bot_to_shoulder_yaw_motor_fxd" trans="0 0.1722 0.256" rpy="0 0 0" parent="bot" child="shoulder_yaw_motor"/>
   <xacro:Revjoint id="shoulder_yaw_joint_rev" trans="0 0 0" rpy="0 0 0" parent="shoulder_yaw_motor" child="shoulder_bracket" axis="0 0 1" l="-3.0357" u="3.24426" v="1.0"/>
@@ -386,6 +387,6 @@
   <xacro:Revjoint id="wrist_pitch" trans="-${length + 0.052 + 0.054} 0 0" rpy="0 0 0" parent="wrist_bracket" child="wrist_pitch_motor" axis="0 0 1" l="-2.36344086" u="2.368556533" v="1.0"/>
   <xacro:FxdJoint id="WP_WY" parent="wrist_pitch_motor" child="wrist_yaw_motor" trans="-0.061 0.02 0" rpy="0 -1.57 0"/>
-  <xacro:Revjoint id="wrist_yaw" trans="0 0 0.065" rpy="-1.57 0 0" parent="wrist_yaw_motor" child="wrist_roll_motor" axis="0 1 0" l="-2.36344086" u="2.368556533" v="1.0"/>
-  <xacro:Revjoint id="wrist_roll" trans="0 0 0" rpy="0 0 0" parent="wrist_roll_motor" child="roll_j_plate" axis="0 0 1" l="-2" u="+2" v="1.0"/>
+  <xacro:Revjoint id="wrist_yaw" trans="0 0 0.065" rpy="0 0 0" parent="wrist_yaw_motor" child="wrist_roll_motor" axis="0 0 1" l="-2.36344086" u="2.368556533" v="1.0"/>
+  <xacro:Revjoint id="wrist_roll" trans="0 0 0" rpy="0 0 1.57" parent="wrist_roll_motor" child="roll_j_plate" axis="1 0 0" l="-2" u="+2" v="1.0"/>
   <xacro:FxdJoint id="roll_plate_gripper" parent="roll_j_plate" child="gripper" trans="0 0 0" rpy="0 0 0"/>
 </robot>

Commit message: Back to 5DOF, libcompute updated planning_using_coordinate script will receive coordinate from kinect and move to that point

File: src/mobile_manipulator/model/mobile_manipulator.urdf (robot description, URDF)
Before this commit: robot mobile_manipulator, 13 links, 12 joints
Joints:
- joint shoulder_yaw: origin xyz=0 0.188 0.2577 rpy=0 0 0 -> xyz=0 0.188 0.2577 rpy=0 0 3.14

File: src/mobile_manipulator/model/mobile_manipulator.xacro (robot description, xacro)
@@ -321,5 +321,5 @@
  <!-- JOINTS -->
   <xacro:FxdJoint id="bot_joint" parent="bot" child="shoulder_yaw_motor"/>
-  <xacro:Revjoint id="shoulder_yaw" trans="0 0.188 0.2577" rpy="0 0 0" parent="shoulder_yaw_motor" child="shoulder_bracket" axis="0 0 1" l="-3.0357" u="3.24426" v="1.0"/>
+  <xacro:Revjoint id="shoulder_yaw" trans="0 0.188 0.2577" rpy="0 0 3.14" parent="shoulder_yaw_motor" child="shoulder_bracket" axis="0 0 1" l="-3.0357" u="3.24426" v="1.0"/>
   <!-- 0 0 0.025 -->
   <xacro:Revjoint id="shoulder_pitch" trans="0 0 0.035" rpy="0 0 0" parent="shoulder_bracket" child="shoulder_pitch_motor" axis="1 0 0" l="-1.973232422" u="1.916503906" v="1.0"/>
